File: Electrical/COTS Prototype/COTS Prototype.kicad_pcb (KiCad board)
At the start: 2 copper layers, 5 parts, among them J301 Raspberry_Pi_2_3, U201 MCP73831-2-OT, U202 TPS61090

Commit message: working on schematics
Parts:
- removed Logo101: SquashedFlyLogo, SquashedFly Logo:SquashedFlyBrightCopper
- added D1: Orange, LED_SMD:LED_0805_2012Metric_Pad1.15x1.40mm_HandSolder, F.Cu at (170.7, 73.0)
- added D2: Green, LED_SMD:LED_0805_2012Metric_Pad1.15x1.40mm_HandSolder, F.Cu at (170.7, 76.1)
- added D4: Blue, LED_SMD:LED_0805_2012Metric_Pad1.15x1.40mm_HandSolder, F.Cu at (175.5, 73.0)
- added Logo1: SquashedFlyLogo, SquashedFly Logo:SquashedFlyBrightCopper, F.Cu at (228.2, 126.2)
- added R1: 10k, Resistor_SMD:R_0603_1608Metric_Pad0.98x0.95mm_HandSolder, F.Cu at (170.4, 78.8)
- added R10: 1k, Resistor_SMD:R_0603_1608Metric_Pad0.98x0.95mm_HandSolder, F.Cu at (183.9, 75.3)
- added R11: 1k5, Resistor_SMD:R_0603_1608Metric_Pad0.98x0.95mm_HandSolder, F.Cu at (193.4, 72.8)
- added R12: 3k3, Resistor_SMD:R_0603_1608Metric_Pad0.98x0.95mm_HandSolder, F.Cu at (193.4, 75.3)
- added R2: 470, Resistor_SMD:R_0603_1608Metric_Pad0.98x0.95mm_HandSolder, F.Cu at (175.2, 75.8)
- added R3: 2k, Resistor_SMD:R_0603_1608Metric_Pad0.98x0.95mm_HandSolder, F.Cu at (180.0, 72.8)
- added R4: 1k, Resistor_SMD:R_0603_1608Metric_Pad0.98x0.95mm_HandSolder, F.Cu at (170.4, 81.3)
- added R5: 10k, Resistor_SMD:R_0603_1608Metric_Pad0.98x0.95mm_HandSolder, F.Cu at (174.8, 78.8)
- added R6: 1M85, Resistor_SMD:R_0603_1608Metric_Pad0.98x0.95mm_HandSolder, F.Cu at (179.6, 75.8)
- added R7: 1M37, Resistor_SMD:R_0603_1608Metric_Pad0.98x0.95mm_HandSolder, F.Cu at (184.4, 72.8)
- added R8: 340k, Resistor_SMD:R_0603_1608Metric_Pad0.98x0.95mm_HandSolder, F.Cu at (174.8, 81.3)
- added R9: 200k, Resistor_SMD:R_0603_1608Metric_Pad0.98x0.95mm_HandSolder, F.Cu at (179.1, 78.3)
- moved U1 17.3 mm to (195.5, 129.0)
- moved U2 12.7 mm to (184.2, 125.2)
- renumbered A301 to A1, J301 to J3, U201 to U1, U202 to U2
Connections:
- A1 pad 16: (no net) -> uC_TX
- A1 pad 28: (no net) -> On_Charge?
- J3 pad 10: (no net) -> RPi_RX
- U1 pad 1: (no net) -> Net-(D1-Pad1)
- U1 pad 4: (no net) -> Supply_+Ve
- U1 pad 5: (no net) -> Net-(R3-Pad1)
- U2 pad 14: (no net) -> Net-(R6-Pad2)
- U2 pad 9: (no net) -> Net-(R7-Pad2)
Other:
- board outline added: 100 x 80 mm

Commit message: working on schematics
Parts:
- added mouse-bite-3mm-slot: VAL**, Panelization:mouse-bite-3mm-slot, F.Cu at (231.0, 78.2)
- added mouse-bite-3mm-slot: VAL**, Panelization:mouse-bite-3mm-slot, F.Cu at (175.5, 78.2)
- moved D1 53.6 mm to (201.7, 116.8)
- moved D2 53.6 mm to (201.7, 119.8)
- moved D4 53.6 mm to (206.5, 116.8)
- moved R1 53.6 mm to (201.4, 122.6)
- moved R10 53.6 mm to (214.9, 119.0)
- moved R11 53.6 mm to (224.4, 116.5)
- moved R12 53.6 mm to (224.4, 119.0)
- moved R2 53.6 mm to (206.2, 119.5)
- moved R3 53.6 mm to (211.0, 116.5)
- moved R4 53.6 mm to (201.4, 125.1)
- moved R5 53.6 mm to (205.8, 122.6)
- moved R6 53.6 mm to (210.6, 119.5)
- moved R7 53.6 mm to (215.4, 116.5)
- moved R8 53.6 mm to (205.8, 125.1)
- moved R9 53.6 mm to (210.1, 122.1)
Routing:
- net RPi_to_uC: track 18.1 -> 0.00 mm
Other:
- board size 100 x 80 mm -> 100 x 117 mm

Commit message: changed COTs PCB
Parts:
- removed the mouse-bite-3mm-slot at (231.0, 78.2)
- removed the mouse-bite-3mm-slot at (175.5, 78.2)
- added mouse-bite-3mm-slot: VAL**, Panelization:mouse-bite-3mm-slot, F.Cu at (176.2, 148.2)
- added mouse-bite-3mm-slot: VAL**, Panelization:mouse-bite-3mm-slot, F.Cu at (127.8, 116.5)
- added mouse-bite-3mm-slot: VAL**, Panelization:mouse-bite-3mm-slot, F.Cu at (127.8, 76.5)
- added mouse-bite-3mm-slot-3way: VAL**, Panelization:mouse-bite-3mm-slot-3way, F.Cu at (148.5, 148.2)
- added mouse-bite-3mm-slot-3way: VAL**, Panelization:mouse-bite-3mm-slot-3way, F.Cu at (127.8, 148.2)
- moved A1 81.2 mm to (134.8, 109.8), turned to 90 degrees
- moved Logo1 44.6 mm to (186.8, 142.5), turned to 90 degrees
- moved U2 37.8 mm to (213.0, 149.8), turned to 90 degrees
- moved J3 33.3 mm to (190.5, 82.4), turned to 180 degrees
- moved U1 23.3 mm to (216.8, 138.5), turned to 90 degrees
- moved R11 21.3 mm to (204.3, 109.6), turned to 90 degrees
- moved R12 20.0 mm to (206.8, 109.6), turned to 90 degrees
- moved D1 15.8 mm to (204.5, 132.3), turned to 90 degrees
- moved D2 13.8 mm to (207.6, 132.3), turned to 90 degrees
- moved R4 13.7 mm to (212.8, 132.6), turned to 90 degrees
- moved R1 13.4 mm to (210.3, 132.6), turned to 90 degrees
- moved R7 11.3 mm to (204.3, 118.6), turned to 90 degrees
- moved D4 10.9 mm to (204.5, 127.5), turned to 90 degrees
- moved R3 9.36 mm to (204.3, 123.0), turned to 90 degrees
- moved R2 8.31 mm to (207.3, 127.8), turned to 90 degrees
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Other:
- board size 100 x 117 mm -> 100 x 100 mm

Commit message: made some changes
Parts:
- removed mouse-bite-3mm-slot (x3): VAL**, Panelization:mouse-bite-3mm-slot
- removed mouse-bite-3mm-slot-3way (x2): VAL**, Panelization:mouse-bite-3mm-slot-3way
- added J1: Battery, Connector_JST:JST_EH_B2B-EH-A_1x02_P2.50mm_Vertical, B.Cu at (134.8, 143.0)
- added J2: Charger, Connector_JST:JST_EH_B3B-EH-A_1x03_P2.50mm_Vertical, F.Cu at (139.5, 143.0)
- moved U1 75.0 mm to (141.8, 137.4)
- moved R3 68.3 mm to (137.5, 137.4), turned to 270 degrees
- moved U2 66.5 mm to (148.0, 135.8), turned to 0 degrees
- moved R1 57.0 mm to (153.6, 137.5), turned to 180 degrees
- moved R2 50.0 mm to (159.0, 140.8), turned to 0 degrees
- moved R4 49.9 mm to (163.6, 140.8), turned to 180 degrees
- moved D1 46.9 mm to (159.0, 143.8), turned to 0 degrees
- moved D2 45.5 mm to (163.5, 143.8), turned to 0 degrees
- moved R10 44.3 mm to (168.2, 140.8), turned to 180 degrees
- moved D4 39.9 mm to (168.0, 143.8), turned to 0 degrees
Connections:
- net Supply_-Ve renamed GND
Routing:
- net Supply_+Ve: track 0.00 -> 21.1 mm
- net Net-(D1-Pad1): track 0.00 -> 16.2 mm
- net Bat_+Ve: track 0.00 -> 16.1 mm
- net Net-(R3-Pad1): track 0.00 -> 3.43 mm
- net Net-(D4-Pad1): track 0.00 -> 3.10 mm
- net Net-(D2-Pad1): track 0.00 -> 3.07 mm
- net Net-(D1-Pad2): track 0.00 -> 3.06 mm
