File: Electrical/COTS Prototype/COTS Prototype.sch (KiCad schematic (older format))
At the start: 1 part

Commit message: working on schematics
Parts:
- removed Logo101: SquashedFlyLogo, SquashedFly Logo:SquashedFlyBrightCopper, symbol SquashedFly_Logo:SquashedFlyLogo
- added Logo1: SquashedFlyLogo, SquashedFly Logo:SquashedFlyBrightCopper, symbol SquashedFly_Logo:SquashedFlyLogo
Changed lines of the file:
@@
 Sheet 1 3
 Title "COTS Swarmbot"
-Date "2021-06-04"
+Date "2021-06-07"
 Rev ""
-Comp "SquashedFly Ltd"
+Comp "{fly} SquashedFly Ltd"
 Comment1 ""
 Comment2 ""
@@
 Comment4 ""
 $EndDescr
-$Comp
-L SquashedFly_Logo:SquashedFlyLogo Logo101
-U 1 1 5E5C26E8
-P 11000 7750
-F 0 "Logo101" H 11000 7850 50  0001 C CNN
-F 1 "SquashedFlyLogo" H 11000 7650 50  0001 C CNN
-F 2 "SquashedFly Logo:SquashedFlyBrightCopper" H 11000 7750 50  0001 C CNN
-F 3 "" H 11000 7750 50  0001 C CNN
-	1    11000 7750
-	1    0    0    -1
-$EndComp
 $Sheet
 S 8100 3500 1550 650
@@
 F1 "MicroControler and RPi Zero.sch" 50
 $EndSheet
+$Comp
+L SquashedFly_Logo:SquashedFlyLogo Logo1
+U 1 1 60BDF508
+P 11000 7750
+F 0 "Logo1" H 11000 7850 50  0001 C CNN
+F 1 "SquashedFlyLogo" H 11000 7650 50  0001 C CNN
+F 2 "SquashedFly Logo:SquashedFlyBrightCopper" H 11000 7750 50  0001 C CNN
+F 3 "~" H 11000 7750 50  0001 C CNN
+	1    11000 7750
+	1    0    0    -1
+$EndComp
+$Comp
+L Graphic:Logo_Open_Hardware_Small #LOGO1
+U 1 1 60BE0501
+P 10700 7100
+F 0 "#LOGO1" H 10700 7375 50  0001 C CNN
+F 1 "Logo_Open_Hardware_Small" H 10700 6875 50  0001 C CNN
+F 2 "Symbol:OSHW-Logo2_14.6x12mm_Copper" H 10700 7100 50  0001 C CNN
+F 3 "~" H 10700 7100 50  0001 C CNN
+	1    10700 7100
+	1    0    0    -1
+$EndComp
 $EndSCHEMATC

Commit message: made some changes
Changed lines of the file:
@@
 $Descr A4 11693 8268
 encoding utf-8
-Sheet 1 3
+Sheet 1 4
 Title "COTS Swarmbot"
 Date "2021-06-07"
@@
 	1    0    0    -1
 $EndComp
+$Sheet
+S 3850 4050 2450 900
+U 60DF275F
+F0 "Minimal STM32" 50
+F1 "Minimal STM32.sch" 50
+$EndSheet
 $EndSCHEMATC
