File: Electrical/COTS Prototype/MicroControler and RPi Zero.sch (KiCad schematic (older format))
At the start: 5 parts, among them J301 Raspberry_Pi_2_3, U301 MIC94052YC6-TR

Commit message: working on schematics
Parts:
- R11: renamed from R301; footprint (none) -> Resistor_SMD:R_0603_1608Metric_Pad0.98x0.95mm_HandSolder
- R12: renamed from R302; footprint (none) -> Resistor_SMD:R_0603_1608Metric_Pad0.98x0.95mm_HandSolder
- renumbered A301 to A1, J301 to J3, U301 to U3
Changed lines of the file:
@@
 $EndDescr
 $Comp
-L MCU_Module:Arduino_UNO_R3 A301
+L MCU_Module:Arduino_UNO_R3 A1
 U 1 1 60BA13E5
 P 2950 2750
-F 0 "A301" H 2950 3931 50  0000 C CNN
+F 0 "A1" H 2950 3931 50  0000 C CNN
 F 1 "Arduino_UNO_R3" H 2950 3840 50  0000 C CNN
 F 2 "Module:Arduino_UNO_R3_WithMountingHoles" H 2950 2750 50  0001 C CIN
@@
 $EndComp
 $Comp
-L Connector:Raspberry_Pi_2_3 J301
+L Connector:Raspberry_Pi_2_3 J3
 U 1 1 60BA3E05
 P 5900 3050
-F 0 "J301" H 5900 4531 50  0000 C CNN
+F 0 "J3" H 5900 4531 50  0000 C CNN
 F 1 "Raspberry_Pi_2_3" H 5900 4440 50  0000 C CNN
 F 2 "Module:Raspberry_Pi_Zero_Socketed_THT_FaceDown_MountingHoles" H 5900 3050 50  0001 C CNN
@@
 $EndComp
 $Comp
-L power:GND #PWR0304
+L power:GND #PWR024
 U 1 1 60BA5BB0
 P 2950 4450
-F 0 "#PWR0304" H 2950 4200 50  0001 C CNN
+F 0 "#PWR024" H 2950 4200 50  0001 C CNN
 F 1 "GND" H 2955 4277 50  0000 C CNN
 F 2 "" H 2950 4450 50  0001 C CNN
@@
 $EndComp
 $Comp
-L power:GND #PWR0305
+L power:GND #PWR025
 U 1 1 60BA6A0F
 P 5500 4450
-F 0 "#PWR0305" H 5500 4200 50  0001 C CNN
+F 0 "#PWR025" H 5500 4200 50  0001 C CNN
 F 1 "GND" H 5505 4277 50  0000 C CNN
 F 2 "" H 5500 4450 50  0001 C CNN
@@
 $EndComp
 $Comp
-L power:GND #PWR0306
+L power:GND #PWR026
 U 1 1 60BA7009
 P 6200 4450
-F 0 "#PWR0306" H 6200 4200 50  0001 C CNN
+F 0 "#PWR026" H 6200 4200 50  0001 C CNN
 F 1 "GND" H 6205 4277 50  0000 C CNN
 F 2 "" H 6200 4450 50  0001 C CNN
@@
 	2300 2250 2450 2250
 $Comp
-L Device:R_Small R301
+L Device:R_Small R11
 U 1 1 60BAB94E
 P 8150 2350
-F 0 "R301" H 8209 2396 50  0000 L CNN
+F 0 "R11" H 8209 2396 50  0000 L CNN
 F 1 "1k5" H 8209 2305 50  0000 L CNN
-F 2 "" H 8150 2350 50  0001 C CNN
+F 2 "Resistor_SMD:R_0603_1608Metric_Pad0.98x0.95mm_HandSolder" H 8150 2350 50  0001 C CNN
 F 3 "~" H 8150 2350 50  0001 C CNN
 	1    8150 2350
@@
 $EndComp
 $Comp
-L Device:R_Small R302
+L Device:R_Small R12
 U 1 1 60BABB80
 P 8150 2750
-F 0 "R302" H 8209 2796 50  0000 L CNN
+F 0 "R12" H 8209 2796 50  0000 L CNN
 F 1 "3k3" H 8209 2705 50  0000 L CNN
-F 2 "" H 8150 2750 50  0001 C CNN
+F 2 "Resistor_SMD:R_0603_1608Metric_Pad0.98x0.95mm_HandSolder" H 8150 2750 50  0001 C CNN
 F 3 "~" H 8150 2750 50  0001 C CNN
 	1    8150 2750
@@
 RPi_RX
 $Comp
-L power:GND #PWR0303
+L power:GND #PWR023
 U 1 1 60BAC2CC
 P 8150 2950
-F 0 "#PWR0303" H 8150 2700 50  0001 C CNN
+F 0 "#PWR023" H 8150 2700 50  0001 C CNN
 F 1 "GND" H 8155 2777 50  0000 C CNN
 F 2 "" H 8150 2950 50  0001 C CNN
@@
 Pi_Power
 $Comp
-L power:+5V #PWR0301
+L power:+5V #PWR021
 U 1 1 60BE2A55
 P 3150 1400
-F 0 "#PWR0301" H 3150 1250 50  0001 C CNN
+F 0 "#PWR021" H 3150 1250 50  0001 C CNN
 F 1 "+5V" H 3165 1573 50  0000 C CNN
 F 2 "" H 3150 1400 50  0001 C CNN
@@
 	3150 1750 3150 1400
 $Comp
-L power:+5V #PWR0302
+L power:+5V #PWR022
 U 1 1 60BE39D3
 P 9250 1900
-F 0 "#PWR0302" H 9250 1750 50  0001 C CNN
+F 0 "#PWR022" H 9250 1750 50  0001 C CNN
 F 1 "+5V" H 9265 2073 50  0000 C CNN
 F 2 "" H 9250 1900 50  0001 C CNN
@@
 $EndComp
 $Comp
-L MIC94052YC6-TR:MIC94052YC6-TR U301
+L MIC94052YC6-TR:MIC94052YC6-TR U3
 U 1 1 60BA5138
 P 9750 2550
-F 0 "U301" H 10228 2558 50  0000 L CNN
+F 0 "U3" H 10228 2558 50  0000 L CNN
 F 1 "MIC94052YC6-TR" H 10228 2467 50  0000 L CNN
 F 2 "" H 9550 2550 50  0001 C CNN
