File: Electrical/COTS Prototype/PowerBoost 500C.sch (KiCad schematic (older format))
At the start: 26 parts, among them J201 Battery, J202 Charger, SW201 SW_SPST, U201 MCP73831-2-OT, U202 TPS61090

Commit message: working on schematics
Parts:
- D1: renamed from D201; footprint (none) -> LED_SMD:LED_0805_2012Metric_Pad1.15x1.40mm_HandSolder
- D2: renamed from D202; footprint (none) -> LED_SMD:LED_0805_2012Metric_Pad1.15x1.40mm_HandSolder
- D4: renamed from D204; footprint (none) -> LED_SMD:LED_0805_2012Metric_Pad1.15x1.40mm_HandSolder
- R1: renamed from R201; footprint (none) -> Resistor_SMD:R_0603_1608Metric_Pad0.98x0.95mm_HandSolder
- R10: renamed from R210; footprint (none) -> Resistor_SMD:R_0603_1608Metric_Pad0.98x0.95mm_HandSolder
- R2: renamed from R202; footprint (none) -> Resistor_SMD:R_0603_1608Metric_Pad0.98x0.95mm_HandSolder
- R3: renamed from R203; footprint (none) -> Resistor_SMD:R_0603_1608Metric_Pad0.98x0.95mm_HandSolder
- R4: renamed from R204; footprint (none) -> Resistor_SMD:R_0603_1608Metric_Pad0.98x0.95mm_HandSolder
- R5: renamed from R205; footprint (none) -> Resistor_SMD:R_0603_1608Metric_Pad0.98x0.95mm_HandSolder
- R6: renamed from R206; footprint (none) -> Resistor_SMD:R_0603_1608Metric_Pad0.98x0.95mm_HandSolder
- R7: renamed from R207; footprint (none) -> Resistor_SMD:R_0603_1608Metric_Pad0.98x0.95mm_HandSolder
- R8: renamed from R208; footprint (none) -> Resistor_SMD:R_0603_1608Metric_Pad0.98x0.95mm_HandSolder
- R9: renamed from R209; footprint (none) -> Resistor_SMD:R_0603_1608Metric_Pad0.98x0.95mm_HandSolder
- renumbered C201 to C1, C202 to C2, C203 to C3, C204 to C4, C205 to C5, C206 to C6, D203 to D3, J201 to J1, J202 to J2, L201 to L1, SW201 to SW1, U201 to U1, U202 to U2

Commit message: made some changes
Parts:
- J1: footprint (none) -> Connector_JST:JST_EH_B2B-EH-A_1x02_P2.50mm_Vertical
- J2: footprint (none) -> Connector_JST:JST_EH_B3B-EH-A_1x03_P2.50mm_Vertical
Changed lines of the file:
@@
 $Descr A4 11693 8268
 encoding utf-8
-Sheet 2 3
+Sheet 2 4
 Title "COTS Swarmbot"
 Date "2021-06-04"
@@
 F 0 "J2" H 1468 825 50  0000 C CNN
 F 1 "Charger" H 1468 916 50  0000 C CNN
-F 2 "" H 1550 1150 50  0001 C CNN
+F 2 "Connector_JST:JST_EH_B3B-EH-A_1x03_P2.50mm_Vertical" H 1550 1150 50  0001 C CNN
 F 3 "~" H 1550 1150 50  0001 C CNN
 	1    1550 1150
@@
 F 0 "J1" H 4380 1042 50  0000 L CNN
 F 1 "Battery" H 4380 951 50  0000 L CNN
-F 2 "" H 4300 1050 50  0001 C CNN
+F 2 "Connector_JST:JST_EH_B2B-EH-A_1x02_P2.50mm_Vertical" H 4300 1050 50  0001 C CNN
 F 3 "~" H 4300 1050 50  0001 C CNN
 	1    4300 1050
@@
 	3900 1450 3900 1150
 Text GLabel 4200 1600 2    50   Output ~ 0
-Supply_-Ve
+GND
 $Comp
 L power:GND #PWR06
