File: Electrical/Swarmbot/Lower PCB.kicad_sch (KiCad schematic)
At the start: 20 parts, among them SW1 Left, SW2 Right, U1 QRE1113GR, U2 QRE1113GR, U3 QRE1113GR, U4 QRE1113GR

Commit message: some little changes have been made
Parts:
- added C25: 100pF, Capacitor_SMD:C_0805_2012Metric_Pad1.18x1.45mm_HandSolder, symbol Device:C_Small
- added R33: 470, Resistor_SMD:R_0805_2012Metric_Pad1.20x1.40mm_HandSolder, symbol Device:R_Small
- added R34: 10k, Resistor_SMD:R_0805_2012Metric_Pad1.20x1.40mm_HandSolder, symbol Device:R_Small
- added Sonar1: Conn_01x04_Male, Connector_PinHeader_2.54mm:PinHeader_1x04_P2.54mm_Vertical, symbol Connector:Conn_01x04_Male
- added U12: QRE1113GR, OptoDevice:OnSemi_CASE100CY, symbol Sensor_Proximity:QRE1113GR
Connections:
- net Line Sensor LEDs: now also R33.1
- net Lower PCB GND: now also U12.2 (K), U12.4
- net Lower PCB Power: now also R34.1
- new net: R33.2, U12.1 (A)
- new net GND: C25.2, Sonar1.4 (Pin_4)
- new net Line Sensor 5: R34.2, U12.3
- new net Sonar 5V: C25.1, Sonar1.1 (Pin_1)
- new net Sonar Echo: Sonar1.3 (Pin_3)
- new net Sonar Trigger: Sonar1.2 (Pin_2)
Other:
- moved on the sheet: C18, C19, H1, H2, R1, R2, R28, R29, R3, R30, R4, R5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

Commit message: some little changes have been made
Parts:
- Sonar1: footprint Connector_PinHeader_2.54mm:PinHeader_1x04_P2.54mm_Vertical -> Connector_PinSocket_2.54mm:PinSocket_1x04_P2.54mm_Vertical
Changed lines of the file:
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@@
       (effects (font (size 1.27 1.27)) (justify right))
     )
-    (property "Footprint" "Connector_PinHeader_2.54mm:PinHeader_1x04_P2.54mm_Vertical" (id 2) (at 241.3 49.53 0)
+    (property "Footprint" "Connector_PinSocket_2.54mm:PinSocket_1x04_P2.54mm_Vertical" (id 2) (at 241.3 49.53 0)
       (effects (font (size 1.27 1.27)) hide)
     )

Commit message: Made some Changes
Parts:
- added R35, R36: 470, Resistor_SMD:R_0805_2012Metric_Pad1.20x1.40mm_HandSolder, symbol Device:R_Small
- added R37, R38: 10k, Resistor_SMD:R_0805_2012Metric_Pad1.20x1.40mm_HandSolder, symbol Device:R_Small
- added U13, U14: TCST2103, TCST2202, TCST2300, symbol Sensor_Proximity:QRE1113GR
- renumbered C18 to C1, C19 to C2, C25 to C3, R29 to R10, R30 to R11, R34 to R12, R33 to R7, R7 to R8, R28 to R9, U12 to U5
Connections:
- net GND is gone; now on net Lower PCB GND: C3.2, Sonar1.4 (Pin_4)
- net Lower PCB GND: now also U13.2 (K), U13.4, U14.2 (K), U14.4
- net Lower PCB Power renamed Lower PCB 3V3
- net Lower PCB 3V3: now also R35.1, R36.1, R37.1, R38.1
- net Sonar 5V renamed Lower PCB 5V
- new net: R35.2, U13.1 (A)
- new net: R36.2, U14.1 (A)
- new net Motor Sensor 1: R37.2, U13.3
- new net Motor Sensor 2: R38.2, U14.3
Other:
- added sheet Motors (Motors.kicad_sch)
- moved on the sheet: C1, C2, H1, H2, R1, R10, R11, R12, R2, R3, R4, R5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
