File: Electrical/Swarmbot/RPi.kicad_sch (KiCad schematic)
At the start: 3 parts, among them J5 Raspberry_Pi_2_3

Commit message: Made some Changes
Parts:
- renumbered C16 to C25, C17 to C26
Changed lines of the file:
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@@
   (symbol (lib_id "power:GND") (at 63.5 68.58 0) (unit 1)
     (in_bom yes) (on_board yes)
-    (property "Reference" "#PWR052" (id 0) (at 63.5 74.93 0)
+    (property "Reference" "#PWR068" (id 0) (at 63.5 74.93 0)
       (effects (font (size 1.27 1.27)) hide)
     )
@@
   (symbol (lib_id "power:GND") (at 76.2 68.58 0) (unit 1)
     (in_bom yes) (on_board yes)
-    (property "Reference" "#PWR053" (id 0) (at 76.2 74.93 0)
+    (property "Reference" "#PWR069" (id 0) (at 76.2 74.93 0)
       (effects (font (size 1.27 1.27)) hide)
     )
@@
   (symbol (lib_id "power:GND") (at 137.16 123.19 0) (unit 1)
     (in_bom yes) (on_board yes) (fields_autoplaced)
-    (property "Reference" "#PWR054" (id 0) (at 137.16 129.54 0)
+    (property "Reference" "#PWR070" (id 0) (at 137.16 129.54 0)
       (effects (font (size 1.27 1.27)) hide)
     )
@@
   (symbol (lib_id "Device:C_Small") (at 63.5 62.23 0) (unit 1)
     (in_bom yes) (on_board yes) (fields_autoplaced)
-    (property "Reference" "C16" (id 0) (at 66.04 60.9599 0)
+    (property "Reference" "C25" (id 0) (at 66.04 60.9599 0)
       (effects (font (size 1.27 1.27)) (justify left))
     )
@@
   (symbol (lib_id "Device:C_Small") (at 76.2 62.23 0) (unit 1)
     (in_bom yes) (on_board yes) (fields_autoplaced)
-    (property "Reference" "C17" (id 0) (at 78.74 60.9599 0)
+    (property "Reference" "C26" (id 0) (at 78.74 60.9599 0)
       (effects (font (size 1.27 1.27)) (justify left))
     )
