File: Electrical/Swarmbot/Top PCB.kicad_sch (KiCad schematic)
At the start: 0 parts

Commit message: some little changes have been made
Parts:
- added Servo1: Conn_01x03_Male, Connector_PinHeader_2.54mm:PinHeader_1x03_P2.54mm_Vertical, symbol Connector:Conn_01x03_Male
Connections:
- net ESP32/Pen Servo: now also Servo1.3 (Pin_3)
- new net +5V: Servo1.2 (Pin_2)
- new net GND: Servo1.1 (Pin_1)
Changed lines of the file:
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@@
     (stroke (width 0) (type default) (color 0 0 0 0))
   )
-  (wire (pts (xy 86.36 97.79) (xy 93.98 97.79))
-    (stroke (width 0) (type default) (color 0 0 0 0))
-  )
-  (wire (pts (xy 86.36 100.33) (xy 93.98 100.33))
-    (stroke (width 0) (type default) (color 0 0 0 0))
-  )
-  (wire (pts (xy 86.36 102.87) (xy 93.98 102.87))
-    (stroke (width 0) (type default) (color 0 0 0 0))
-  )
-  (wire (pts (xy 86.36 105.41) (xy 93.98 105.41))
+  (wire (pts (xy 86.36 85.09) (xy 130.175 85.09))
+    (stroke (width 0) (type default) (color 0 0 0 0))
+  )
+  (wire (pts (xy 86.36 91.44) (xy 93.98 91.44))
+    (stroke (width 0) (type default) (color 0 0 0 0))
+  )
+  (wire (pts (xy 86.36 93.98) (xy 93.98 93.98))
+    (stroke (width 0) (type default) (color 0 0 0 0))
+  )
+  (wire (pts (xy 86.36 100.965) (xy 93.98 100.965))
+    (stroke (width 0) (type default) (color 0 0 0 0))
+  )
+  (wire (pts (xy 86.36 103.505) (xy 93.98 103.505))
+    (stroke (width 0) (type default) (color 0 0 0 0))
+  )
+  (wire (pts (xy 86.36 106.045) (xy 93.98 106.045))
+    (stroke (width 0) (type default) (color 0 0 0 0))
+  )
+  (wire (pts (xy 86.36 108.585) (xy 93.98 108.585))
+    (stroke (width 0) (type default) (color 0 0 0 0))
+  )
+  (wire (pts (xy 128.27 87.63) (xy 128.27 82.55))
+    (stroke (width 0) (type default) (color 0 0 0 0))
+  )
+  (wire (pts (xy 128.27 90.17) (xy 128.27 92.075))
+    (stroke (width 0) (type default) (color 0 0 0 0))
+  )
+  (wire (pts (xy 128.27 90.17) (xy 130.175 90.17))
+    (stroke (width 0) (type default) (color 0 0 0 0))
+  )
+  (wire (pts (xy 130.175 87.63) (xy 128.27 87.63))
     (stroke (width 0) (type default) (color 0 0 0 0))
   )
@@
     (effects (font (size 1.27 1.27)) (justify left))
   )
-  (sheet (at 58.42 26.67) (size 27.94 90.17) (fields_autoplaced)
+  (hierarchical_label "Sonar Trigger" (shape output) (at 93.98 91.44 0)
+    (effects (font (size 1.27 1.27)) (justify left))
+  )
+  (hierarchical_label "Sonar Echo" (shape input) (at 93.98 93.98 0)
+    (effects (font (size 1.27 1.27)) (justify left))
+  )
+  (symbol (lib_id "power:+5V") (at 128.27 82.55 0) (unit 1)
+    (in_bom yes) (on_board yes) (fields_autoplaced)
+    (property "Reference" "#PWR0109" (id 0) (at 128.27 86.36 0)
+      (effects (font (size 1.27 1.27)) hide)
+    )
+    (property "Value" "+5V" (id 1) (at 128.27 77.47 0))
+    (property "Footprint" "" (id 2) (at 128.27 82.55 0)
+      (effects (font (size 1.27 1.27)) hide)
+    )
+    (property "Datasheet" "" (id 3) (at 128.27 82.55 0)
+      (effects (font (size 1.27 1.27)) hide)
+    )
+    (pin "1")
+  )
+  (symbol (lib_id "power:GND") (at 128.27 92.075 0) (unit 1)
+    (in_bom yes) (on_board yes) (fields_autoplaced)
+    (property "Reference" "#PWR0111" (id 0) (at 128.27 98.425 0)
+      (effects (font (size 1.27 1.27)) hide)
+    )
+    (property "Value" "GND" (id 1) (at 128.27 97.155 0))
+    (property "Footprint" "" (id 2) (at 128.27 92.075 0)
+      (effects (font (size 1.27 1.27)) hide)
+    )
+    (property "Datasheet" "" (id 3) (at 128.27 92.075 0)
+      (effects (font (size 1.27 1.27)) hide)
+    )
+    (pin "1")
+  )
+  (symbol (lib_id "Connector:Conn_01x03_Male") (at 135.255 87.63 180) (unit 1)
+    (in_bom yes) (on_board yes)
+    (property "Reference" "Servo1" (id 0) (at 136.525 86.3599 0)
+      (effects (font (size 1.27 1.27)) (justify right))
+    )
+    (property "Value" "Conn_01x03_Male" (id 1) (at 136.525 88.8999 0)
+      (effects (font (size 1.27 1.27)) (justify right))
+    )
+    (property "Footprint" "Connector_PinHeader_2.54mm:PinHeader_1x03_P2.54mm_Vertical" (id 2) (at 135.255 87.63 0)
+      (effects (font (size 1.27 1.27)) hide)
+    )
+    (property "Datasheet" "~" (id 3) (at 135.255 87.63 0)
+      (effects (font (size 1.27 1.27)) hide)
+    )
+    (pin "1")
+    (pin "2")
+    (pin "3")
+  )
+  (sheet (at 58.42 26.67) (size 27.94 93.98) (fields_autoplaced)
     (stroke (width 0.1524) (type solid) (color 0 0 0 0))
     (fill (color 0 0 0 0.0000))
@@
       (effects (font (size 1.27 1.27)) (justify left bottom))
     )
-    (property "Sheet file" "ESP32.kicad_sch" (id 1) (at 58.42 117.4246 0)
+    (property "Sheet file" "ESP32.kicad_sch" (id 1) (at 58.42 121.2346 0)
       (effects (font (size 1.27 1.27)) (justify left top))
     )
@@
       (effects (font (size 1.27 1.27)) (justify right))
     )
-    (pin "Motor PWM3" output (at 86.36 102.87 0)
-      (effects (font (size 1.27 1.27)) (justify right))
-    )
-    (pin "Motor PWM2" output (at 86.36 100.33 0)
-      (effects (font (size 1.27 1.27)) (justify right))
-    )
-    (pin "Motor PWM1" output (at 86.36 97.79 0)
-      (effects (font (size 1.27 1.27)) (justify right))
-    )
-    (pin "Motor PWM4" output (at 86.36 105.41 0)
-      (effects (font (size 1.27 1.27)) (justify right))
-    )
-    (pin "Motor Sensor 2" input (at 86.36 111.76 0)
-      (effects (font (size 1.27 1.27)) (justify right))
-    )
-    (pin "Motor Sensor 1" input (at 86.36 109.22 0)
+    (pin "Motor PWM3" output (at 86.36 106.045 0)
+      (effects (font (size 1.27 1.27)) (justify right))
+    )
+    (pin "Motor PWM2" output (at 86.36 103.505 0)
+      (effects (font (size 1.27 1.27)) (justify right))
+    )
+    (pin "Motor PWM1" output (at 86.36 100.965 0)
+      (effects (font (size 1.27 1.27)) (justify right))
+    )
+    (pin "Motor PWM4" output (at 86.36 108.585 0)
+      (effects (font (size 1.27 1.27)) (justify right))
+    )
+    (pin "Motor Sensor 2" input (at 86.36 114.935 0)
+      (effects (font (size 1.27 1.27)) (justify right))
+    )
+    (pin "Motor Sensor 1" input (at 86.36 112.395 0)
       (effects (font (size 1.27 1.27)) (justify right))
     )
@@
       (effects (font (size 1.27 1.27)) (justify right))
     )
-    (pin "Pen Servo" output (at 86.36 87.63 0)
+    (pin "Pen Servo" output (at 86.36 85.09 0)
       (effects (font (size 1.27 1.27)) (justify right))
     )
@@
     )
   )
-  (sheet (at 93.98 95.885) (size 24.13 20.955) (fields_autoplaced)
+  (sheet (at 93.98 99.06) (size 24.13 20.955) (fields_autoplaced)
     (stroke (width 0.1524) (type solid) (color 0 0 0 0))
     (fill (color 0 0 0 0.0000))
-    (property "Sheet name" "Motors" (id 0) (at 93.98 95.1734 0)
+    (property "Sheet name" "Motors" (id 0) (at 93.98 98.3484 0)
       (effects (font (size 1.27 1.27)) (justify left bottom))
     )
-    (property "Sheet file" "Motors.kicad_sch" (id 1) (at 93.98 117.4246 0)
+    (property "Sheet file" "Motors.kicad_sch" (id 1) (at 93.98 120.5996 0)
       (effects (font (size 1.27 1.27)) (justify left top))
     )
-    (pin "IN1A" input (at 93.98 97.79 180)
-      (effects (font (size 1.27 1.27)) (justify left))
-    )
-    (pin "IN1B" input (at 93.98 100.33 180)
-      (effects (font (size 1.27 1.27)) (justify left))
-    )
-    (pin "IN2A" input (at 93.98 102.87 180)
-      (effects (font (size 1.27 1.27)) (justify left))
-    )
-    (pin "IN2B" input (at 93.98 105.41 180)
-      (effects (font (size 1.27 1.27)) (justify left))
-    )
+    (pin "IN1A" input (at 93.98 100.965 180)
+      (effects (font (size 1.27 1.27)) (justify left))
+    )
+    (pin "IN1B" input (at 93.98 103.505 180)
+      (effects (font (size 1.27 1.27)) (justify left))
+    )
+    (pin "IN2A" input (at 93.98 106.045 180)
+      (effects (font (size 1.27 1.27)) (justify left))
+    )
+    (pin "IN2B" input (at 93.98 108.585 180)
+      (effects (font (size 1.27 1.27)) (justify left))
+    )

Commit message: Made some Changes
Other:
- removed sheet Motors
Changed lines of the file:
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@@
+    (stroke (width 0) (type default) (color 0 0 0 0))
+  )
+  (wire (pts (xy 86.36 112.395) (xy 93.98 112.395))
+    (stroke (width 0) (type default) (color 0 0 0 0))
+  )
+  (wire (pts (xy 86.36 114.935) (xy 93.98 114.935))
     (stroke (width 0) (type default) (color 0 0 0 0))
   )
@@
     (effects (font (size 1.27 1.27)) (justify left))
   )
+  (hierarchical_label "H-Bridge 1A" (shape output) (at 93.98 100.965 0)
+    (effects (font (size 1.27 1.27)) (justify left))
+  )
+  (hierarchical_label "H-Bridge 1B" (shape output) (at 93.98 103.505 0)
+    (effects (font (size 1.27 1.27)) (justify left))
+  )
+  (hierarchical_label "H-Bridge 2A" (shape output) (at 93.98 106.045 0)
+    (effects (font (size 1.27 1.27)) (justify left))
+  )
+  (hierarchical_label "H-Bridge 2B" (shape output) (at 93.98 108.585 0)
+    (effects (font (size 1.27 1.27)) (justify left))
+  )
+  (hierarchical_label "Motor Sensor 1" (shape input) (at 93.98 112.395 0)
+    (effects (font (size 1.27 1.27)) (justify left))
+  )
+  (hierarchical_label "Motor Sensor 2" (shape input) (at 93.98 114.935 0)
+    (effects (font (size 1.27 1.27)) (justify left))
+  )
   (symbol (lib_id "power:+5V") (at 128.27 82.55 0) (unit 1)
     (in_bom yes) (on_board yes) (fields_autoplaced)
-    (property "Reference" "#PWR0109" (id 0) (at 128.27 86.36 0)
+    (property "Reference" "#PWR04" (id 0) (at 128.27 86.36 0)
       (effects (font (size 1.27 1.27)) hide)
     )
@@
   (symbol (lib_id "power:GND") (at 128.27 92.075 0) (unit 1)
     (in_bom yes) (on_board yes) (fields_autoplaced)
-    (property "Reference" "#PWR0111" (id 0) (at 128.27 98.425 0)
+    (property "Reference" "#PWR05" (id 0) (at 128.27 98.425 0)
       (effects (font (size 1.27 1.27)) hide)
     )
@@
     )
   )
-  (sheet (at 93.98 99.06) (size 24.13 20.955) (fields_autoplaced)
-    (stroke (width 0.1524) (type solid) (color 0 0 0 0))
-    (fill (color 0 0 0 0.0000))
-    (property "Sheet name" "Motors" (id 0) (at 93.98 98.3484 0)
-      (effects (font (size 1.27 1.27)) (justify left bottom))
-    )
-    (property "Sheet file" "Motors.kicad_sch" (id 1) (at 93.98 120.5996 0)
-      (effects (font (size 1.27 1.27)) (justify left top))
-    )
-    (pin "IN1A" input (at 93.98 100.965 180)
-      (effects (font (size 1.27 1.27)) (justify left))
-    )
-    (pin "IN1B" input (at 93.98 103.505 180)
-      (effects (font (size 1.27 1.27)) (justify left))
-    )
-    (pin "IN2A" input (at 93.98 106.045 180)
-      (effects (font (size 1.27 1.27)) (justify left))
-    )
-    (pin "IN2B" input (at 93.98 108.585 180)
-      (effects (font (size 1.27 1.27)) (justify left))
-    )
-  )
