File: Electrical/Swarmbot/power.kicad_sch (KiCad schematic)
At the start: 39 parts, among them J3 Charging Header, J4 Battery 1S2P, SW3 SW_SPST, U6 TP4056, U7 FP6298, U8 AP9101CK, U9 AP2112K-3.3

Commit message: some little changes have been made
Parts:
- added C26: 100nF, Capacitor_SMD:C_0805_2012Metric_Pad1.18x1.45mm_HandSolder, symbol Device:C_Small
- added R31: .0025R, Resistor_SMD:R_1206_3216Metric_Pad1.30x1.75mm_HandSolder, symbol Device:R_Small
- added R32: 2k7, Resistor_SMD:R_0805_2012Metric_Pad1.20x1.40mm_HandSolder, symbol Device:R_Small
- added U11: INA138, Package_TO_SOT_SMD:SOT-23-5, symbol Amplifier_Current:INA138
Connections:
- net PowerIn is gone; now on net Charging Pad: D2.2 (A), D7.2 (A), J3.1 (Pin_1)
- net +3V3: now also U11.5 (V+)
- net +BATT: now also R31.2, U11.3 (+)
- net Bat I: now also C26.1, R32.1
- net GND: now also C26.2, U11.2 (GND)
- net Bat+VE: now reaches J4.1 (Pin_1), J4.2 (Pin_2)
- net Bat+VE: now also R31.1, U11.4 (-)
- new net: R32.2, U11.1

Commit message: Made some Changes
Parts:
- renumbered C5 to C13, C6 to C14, C7 to C15, C8 to C16, C9 to C17, C10 to C18, C11 to C19, C12 to C20, C13 to C21, C14 to C22, C15 to C23, C26 to C24, R15 to R20, R16 to R21, R17 to R22, R18 to R23, R19 to R24, R20 to R25, R21 to R26, R22 to R27, R23 to R28, R24 to R29, R25 to R30, R26 to R31, R27 to R32, R31 to R33, R32 to R34, U8 to U10, U9 to U11, U11 to U12, U6 to U8, U7 to U9
