File: Electrical/Swarmbot/ESP32.kicad_sch (KiCad schematic)
At the start: 19 parts, among them Q1 BSH108, Q2 BSH108, Q3 BSH108, Q4 BSH108, Q5 RSC002P03, Q6 RSC002P03, U5 ESP32-WROOM-32D

Commit message: some little changes have been made
Connections:
- net Left Switch: now also U5.14 (IO12); no longer U5.13 (IO14)
- net Motor Sensor 1: now also U5.33 (IO21); no longer U5.11 (IO26)
- net Motor Sensor 2: now also U5.36 (IO22); no longer U5.12 (IO27)
- net Right Switch: now also U5.13 (IO14); no longer U5.14 (IO12)
- net Sonar Echo: now also U5.12 (IO27); no longer U5.33 (IO21)
- net Sonar Trigger: now also U5.11 (IO26); no longer U5.36 (IO22)
Changed lines of the file:
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@@
     (effects (font (size 1.27 1.27)) (justify left))
   )
-  (hierarchical_label "Right Switch" (shape input) (at 182.88 59.69 0)
+  (hierarchical_label "Left Switch" (shape input) (at 182.88 59.69 0)
     (effects (font (size 1.27 1.27)) (justify left))
   )
@@
     (effects (font (size 1.27 1.27)) (justify left))
   )
-  (hierarchical_label "Left Switch" (shape input) (at 182.88 64.77 0)
+  (hierarchical_label "Right Switch" (shape input) (at 182.88 64.77 0)
     (effects (font (size 1.27 1.27)) (justify left))
   )
@@
     (effects (font (size 1.27 1.27)) (justify left))
   )
-  (hierarchical_label "Sonar Echo" (shape input) (at 182.88 80.01 0)
+  (hierarchical_label "Motor Sensor 1" (shape input) (at 182.88 80.01 0)
     (effects (font (size 1.27 1.27)) (justify left))
   )
-  (hierarchical_label "Sonar Trigger" (shape output) (at 182.88 82.55 0)
+  (hierarchical_label "Motor Sensor 2" (shape input) (at 182.88 82.55 0)
     (effects (font (size 1.27 1.27)) (justify left))
   )
@@
     (effects (font (size 1.27 1.27)) (justify left))
   )
-  (hierarchical_label "Motor Sensor 1" (shape input) (at 182.88 90.17 0)
+  (hierarchical_label "Sonar Trigger" (shape output) (at 182.88 90.17 0)
     (effects (font (size 1.27 1.27)) (justify left))
   )
-  (hierarchical_label "Motor Sensor 2" (shape input) (at 182.88 92.71 0)
+  (hierarchical_label "Sonar Echo" (shape input) (at 182.88 92.71 0)
     (effects (font (size 1.27 1.27)) (justify left))
   )

Commit message: Made some Changes
Parts:
- renumbered C2 to C10, C3 to C11, C4 to C12, C1 to C9, R8 to R13, R9 to R14, R10 to R15, R11 to R16, R12 to R17, R13 to R18, R14 to R19, U5 to U7
Changed lines of the file:
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@@
   (symbol (lib_id "power:+3V3") (at 64.77 34.29 0) (unit 1)
     (in_bom yes) (on_board yes) (fields_autoplaced)
-    (property "Reference" "#PWR07" (id 0) (at 64.77 38.1 0)
+    (property "Reference" "#PWR020" (id 0) (at 64.77 38.1 0)
       (effects (font (size 1.27 1.27)) hide)
     )
@@
   (symbol (lib_id "power:+3V3") (at 64.77 72.39 0) (unit 1)
     (in_bom yes) (on_board yes) (fields_autoplaced)
-    (property "Reference" "#PWR09" (id 0) (at 64.77 76.2 0)
+    (property "Reference" "#PWR022" (id 0) (at 64.77 76.2 0)
       (effects (font (size 1.27 1.27)) hide)
     )
@@
   (symbol (lib_id "power:+5V") (at 64.77 110.49 0) (unit 1)
     (in_bom yes) (on_board yes) (fields_autoplaced)
-    (property "Reference" "#PWR011" (id 0) (at 64.77 114.3 0)
+    (property "Reference" "#PWR024" (id 0) (at 64.77 114.3 0)
       (effects (font (size 1.27 1.27)) hide)
     )
@@
   (symbol (lib_id "power:+5V") (at 64.77 154.94 0) (unit 1)
     (in_bom yes) (on_board yes) (fields_autoplaced)
-    (property "Reference" "#PWR013" (id 0) (at 64.77 158.75 0)
+    (property "Reference" "#PWR026" (id 0) (at 64.77 158.75 0)
       (effects (font (size 1.27 1.27)) hide)
     )
@@
   (symbol (lib_id "power:+3V3") (at 97.79 34.29 0) (unit 1)
     (in_bom yes) (on_board yes) (fields_autoplaced)
-    (property "Reference" "#PWR017" (id 0) (at 97.79 38.1 0)
+    (property "Reference" "#PWR030" (id 0) (at 97.79 38.1 0)
       (effects (font (size 1.27 1.27)) hide)
     )
@@
   (symbol (lib_id "power:+3V3") (at 116.84 34.29 0) (unit 1)
     (in_bom yes) (on_board yes) (fields_autoplaced)
-    (property "Reference" "#PWR019" (id 0) (at 116.84 38.1 0)
+    (property "Reference" "#PWR032" (id 0) (at 116.84 38.1 0)
       (effects (font (size 1.27 1.27)) hide)
     )
@@
   (symbol (lib_id "power:+3V3") (at 160.02 34.29 0) (unit 1)
     (in_bom yes) (on_board yes) (fields_autoplaced)
-    (property "Reference" "#PWR021" (id 0) (at 160.02 38.1 0)
+    (property "Reference" "#PWR034" (id 0) (at 160.02 38.1 0)
       (effects (font (size 1.27 1.27)) hide)
     )
@@
   (symbol (lib_id "power:+3V3") (at 243.84 34.29 0) (unit 1)
     (in_bom yes) (on_board yes) (fields_autoplaced)
-    (property "Reference" "#PWR023" (id 0) (at 243.84 38.1 0)
+    (property "Reference" "#PWR036" (id 0) (at 243.84 38.1 0)
       (effects (font (size 1.27 1.27)) hide)
     )
@@
   (symbol (lib_id "power:GND") (at 64.77 55.88 0) (unit 1)
     (in_bom yes) (on_board yes) (fields_autoplaced)
-    (property "Reference" "#PWR08" (id 0) (at 64.77 62.23 0)
+    (property "Reference" "#PWR021" (id 0) (at 64.77 62.23 0)
       (effects (font (size 1.27 1.27)) hide)
     )
@@
   (symbol (lib_id "power:GND") (at 64.77 93.98 0) (unit 1)
     (in_bom yes) (on_board yes) (fields_autoplaced)
-    (property "Reference" "#PWR010" (id 0) (at 64.77 100.33 0)
+    (property "Reference" "#PWR023" (id 0) (at 64.77 100.33 0)
       (effects (font (size 1.27 1.27)) hide)
     )
@@
   (symbol (lib_id "power:GND") (at 64.77 138.43 0) (unit 1)
     (in_bom yes) (on_board yes) (fields_autoplaced)
-    (property "Reference" "#PWR012" (id 0) (at 64.77 144.78 0)
+    (property "Reference" "#PWR025" (id 0) (at 64.77 144.78 0)
       (effects (font (size 1.27 1.27)) hide)
     )
@@
   (symbol (lib_id "power:GND") (at 64.77 182.88 0) (unit 1)
     (in_bom yes) (on_board yes) (fields_autoplaced)
-    (property "Reference" "#PWR014" (id 0) (at 64.77 189.23 0)
+    (property "Reference" "#PWR027" (id 0) (at 64.77 189.23 0)
       (effects (font (size 1.27 1.27)) hide)
     )
@@
   (symbol (lib_id "power:GND") (at 81.28 138.557 0) (unit 1)
     (in_bom yes) (on_board yes) (fields_autoplaced)
-    (property "Reference" "#PWR015" (id 0) (at 81.28 144.907 0)
+    (property "Reference" "#PWR028" (id 0) (at 81.28 144.907 0)
       (effects (font (size 1.27 1.27)) hide)
     )
@@
   (symbol (lib_id "power:GND") (at 82.169 183.007 0) (unit 1)
     (in_bom yes) (on_board yes) (fields_autoplaced)
-    (property "Reference" "#PWR016" (id 0) (at 82.169 189.357 0)
+    (property "Reference" "#PWR029" (id 0) (at 82.169 189.357 0)
       (effects (font (size 1.27 1.27)) hide)
     )
@@
   (symbol (lib_id "power:GND") (at 97.79 45.72 0) (unit 1)
     (in_bom yes) (on_board yes)
-    (property "Reference" "#PWR018" (id 0) (at 97.79 52.07 0)
+    (property "Reference" "#PWR031" (id 0) (at 97.79 52.07 0)
       (effects (font (size 1.27 1.27)) hide)
     )
@@
   (symbol (lib_id "power:GND") (at 116.84 45.72 0) (unit 1)
     (in_bom yes) (on_board yes)
-    (property "Reference" "#PWR020" (id 0) (at 116.84 52.07 0)
+    (property "Reference" "#PWR033" (id 0) (at 116.84 52.07 0)
       (effects (font (size 1.27 1.27)) hide)
     )
@@
   (symbol (lib_id "power:GND") (at 160.02 113.03 0) (unit 1)
     (in_bom yes) (on_board yes) (fields_autoplaced)
-    (property "Reference" "#PWR022" (id 0) (at 160.02 119.38 0)
+    (property "Reference" "#PWR035" (id 0) (at 160.02 119.38 0)
       (effects (font (size 1.27 1.27)) hide)
     )
@@
   (symbol (lib_id "power:GND") (at 245.11 52.07 0) (unit 1)
     (in_bom yes) (on_board yes) (fields_autoplaced)
-    (property "Reference" "#PWR024" (id 0) (at 245.11 58.42 0)
+    (property "Reference" "#PWR037" (id 0) (at 245.11 58.42 0)
       (effects (font (size 1.27 1.27)) hide)
     )
@@
   (symbol (lib_id "Device:R_Small") (at 53.34 120.65 90) (unit 1)
     (in_bom yes) (on_board yes) (fields_autoplaced)
-    (property "Reference" "R8" (id 0) (at 53.34 114.3 90))
+    (property "Reference" "R13" (id 0) (at 53.34 114.3 90))
     (property "Value" "10k" (id 1) (at 53.34 116.84 90))
     (property "Footprint" "Resistor_SMD:R_0805_2012Metric_Pad1.20x1.40mm_HandSolder" (id 2) (at 53.34 120.65 0)
@@
   (symbol (lib_id "Device:R_Small") (at 53.34 129.54 90) (unit 1)
     (in_bom yes) (on_board yes) (fields_autoplaced)
-    (property "Reference" "R9" (id 0) (at 53.34 123.19 90))
+    (property "Reference" "R14" (id 0) (at 53.34 123.19 90))
     (property "Value" "10k" (id 1) (at 53.34 125.73 90))
     (property "Footprint" "Resistor_SMD:R_0805_2012Metric_Pad1.20x1.40mm_HandSolder" (id 2) (at 53.34 129.54 0)
@@
   (symbol (lib_id "Device:R_Small") (at 53.34 173.99 90) (unit 1)
     (in_bom yes) (on_board yes) (fields_autoplaced)
-    (property "Reference" "R10" (id 0) (at 53.34 167.64 90))
+    (property "Reference" "R15" (id 0) (at 53.34 167.64 90))
     (property "Value" "10k" (id 1) (at 53.34 170.18 90))
     (property "Footprint" "Resistor_SMD:R_0805_2012Metric_Pad1.20x1.40mm_HandSolder" (id 2) (at 53.34 173.99 0)
@@
   (symbol (lib_id "Device:R_Small") (at 64.77 39.37 0) (unit 1)
     (in_bom yes) (on_board yes) (fields_autoplaced)
-    (property "Reference" "R11" (id 0) (at 67.31 38.0999 0)
+    (property "Reference" "R16" (id 0) (at 67.31 38.0999 0)
       (effects (font (size 1.27 1.27)) (justify left))
     )
@@
   (symbol (lib_id "Device:R_Small") (at 64.77 78.74 0) (unit 1)
     (in_bom yes) (on_board yes) (fields_autoplaced)
-    (property "Reference" "R12" (id 0) (at 67.31 77.4699 0)
+    (property "Reference" "R17" (id 0) (at 67.31 77.4699 0)
       (effects (font (size 1.27 1.27)) (justify left))
     )
@@
   (symbol (lib_id "Device:R_Small") (at 64.77 115.57 0) (unit 1)
     (in_bom yes) (on_board yes) (fields_autoplaced)
-    (property "Reference" "R13" (id 0) (at 67.31 114.2999 0)
+    (property "Reference" "R18" (id 0) (at 67.31 114.2999 0)
       (effects (font (size 1.27 1.27)) (justify left))
     )
@@
   (symbol (lib_id "Device:R_Small") (at 64.77 160.02 0) (unit 1)
     (in_bom yes) (on_board yes) (fields_autoplaced)
-    (property "Reference" "R14" (id 0) (at 67.31 158.7499 0)
+    (property "Reference" "R19" (id 0) (at 67.31 158.7499 0)
       (effects (font (size 1.27 1.27)) (justify left))
     )
@@
   (symbol (lib_id "Device:C_Small") (at 81.28 135.128 0) (unit 1)
     (in_bom yes) (on_board yes) (fields_autoplaced)
-    (property "Reference" "C1" (id 0) (at 83.82 133.8579 0)
+    (property "Reference" "C9" (id 0) (at 83.82 133.8579 0)
       (effects (font (size 1.27 1.27)) (justify left))
     )
@@
   (symbol (lib_id "Device:C_Small") (at 82.169 178.943 0) (unit 1)
     (in_bom yes) (on_board yes) (fields_autoplaced)
-    (property "Reference" "C2" (id 0) (at 84.709 177.6729 0)
+    (property "Reference" "C10" (id 0) (at 84.709 177.6729 0)
       (effects (font (size 1.27 1.27)) (justify left))
     )
@@
   (symbol (lib_id "Device:C_Small") (at 97.79 39.37 0) (unit 1)
     (in_bom yes) (on_board yes) (fields_autoplaced)
-    (property "Reference" "C3" (id 0) (at 100.33 38.0999 0)
+    (property "Reference" "C11" (id 0) (at 100.33 38.0999 0)
       (effects (font (size 1.27 1.27)) (justify left))
     )
@@
   (symbol (lib_id "Device:C_Small") (at 116.84 39.37 0) (unit 1)
     (in_bom yes) (on_board yes) (fields_autoplaced)
-    (property "Reference" "C4" (id 0) (at 119.38 38.0999 0)
+    (property "Reference" "C12" (id 0) (at 119.38 38.0999 0)
       (effects (font (size 1.27 1.27)) (justify left))
     )
@@
   (symbol (lib_id "RF_Module:ESP32-WROOM-32D") (at 160.02 74.93 0) (unit 1)
     (in_bom yes) (on_board yes)
-    (property "Reference" "U5" (id 0) (at 160.02 74.93 0))
+    (property "Reference" "U7" (id 0) (at 160.02 74.93 0))
     (property "Value" "ESP32-WROOM-32D" (id 1) (at 160.02 36.83 0))
     (property "Footprint" "RF_Module:ESP32-WROOM-32" (id 2) (at 160.02 113.03 0)

Commit message: updated the excel
Other:
- note added: "For this sheet, Pin assignment and function please keep in sync with 'Swarmbot IO Assignment.xlsx' in the folder."
- moved on the sheet: ESP1
Changed lines of the file:
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@@
+    (stroke (width 0) (type default) (color 0 0 0 0))
+  )
+  (wire (pts (xy 93.98 80.645) (xy 99.06 80.645))
+    (stroke (width 0) (type default) (color 0 0 0 0))
+  )
+  (wire (pts (xy 93.98 83.185) (xy 99.06 83.185))
+    (stroke (width 0) (type default) (color 0 0 0 0))
+  )
+  (wire (pts (xy 93.98 85.725) (xy 99.06 85.725))
     (stroke (width 0) (type default) (color 0 0 0 0))
   )
@@
     (stroke (width 0) (type default) (color 0 0 0 0))
   )
+  (wire (pts (xy 127 83.185) (xy 133.35 83.185))
+    (stroke (width 0) (type default) (color 0 0 0 0))
+  )
+  (wire (pts (xy 129.54 74.295) (xy 129.54 85.725))
+    (stroke (width 0) (type default) (color 0 0 0 0))
+  )
+  (wire (pts (xy 129.54 85.725) (xy 127 85.725))
+    (stroke (width 0) (type default) (color 0 0 0 0))
+  )
+  (wire (pts (xy 130.81 80.645) (xy 127 80.645))
+    (stroke (width 0) (type default) (color 0 0 0 0))
+  )
+  (wire (pts (xy 130.81 92.075) (xy 130.81 80.645))
+    (stroke (width 0) (type default) (color 0 0 0 0))
+  )
   (wire (pts (xy 137.16 44.45) (xy 144.78 44.45))
     (stroke (width 0) (type default) (color 0 0 0 0))
@@
     (stroke (width 0) (type default) (color 0 0 0 0))
   )
-  (wire (pts (xy 208.28 40.64) (xy 213.36 40.64))
-    (stroke (width 0) (type default) (color 0 0 0 0))
-  )
-  (wire (pts (xy 208.28 43.18) (xy 213.36 43.18))
-    (stroke (width 0) (type default) (color 0 0 0 0))
-  )
-  (wire (pts (xy 208.28 45.72) (xy 213.36 45.72))
-    (stroke (width 0) (type default) (color 0 0 0 0))
-  )
-  (wire (pts (xy 241.3 43.18) (xy 247.65 43.18))
-    (stroke (width 0) (type default) (color 0 0 0 0))
-  )
-  (wire (pts (xy 243.84 34.29) (xy 243.84 45.72))
-    (stroke (width 0) (type default) (color 0 0 0 0))
-  )
-  (wire (pts (xy 243.84 45.72) (xy 241.3 45.72))
-    (stroke (width 0) (type default) (color 0 0 0 0))
-  )
-  (wire (pts (xy 245.11 40.64) (xy 241.3 40.64))
-    (stroke (width 0) (type default) (color 0 0 0 0))
-  )
-  (wire (pts (xy 245.11 52.07) (xy 245.11 40.64))
-    (stroke (width 0) (type default) (color 0 0 0 0))
+  (text "For this sheet, Pin assignment and function please keep in sync with \n'Swarmbot IO Assignment.xlsx' in the folder."
+    (at 185.42 178.435 0)
+    (effects (font (size 1.27 1.27)) (justify left bottom))
   )
   (label "5V Switch 1" (at 49.53 129.54 180)
@@
     (effects (font (size 1.27 1.27)) (justify left))
   )
+  (hierarchical_label "Flash" (shape input) (at 93.98 80.645 180)
+    (effects (font (size 1.27 1.27)) (justify right))
+  )
+  (hierarchical_label "TX" (shape bidirectional) (at 93.98 83.185 180)
+    (effects (font (size 1.27 1.27)) (justify right))
+  )
+  (hierarchical_label "RX" (shape bidirectional) (at 93.98 85.725 180)
+    (effects (font (size 1.27 1.27)) (justify right))
+  )
+  (hierarchical_label "Reset" (shape input) (at 133.35 83.185 0)
+    (effects (font (size 1.27 1.27)) (justify left))
+  )
   (hierarchical_label "TX" (shape bidirectional) (at 182.88 46.99 0)
     (effects (font (size 1.27 1.27)) (justify left))
@@
   )
   (hierarchical_label "Motor PWM3" (shape output) (at 182.88 102.87 0)
-    (effects (font (size 1.27 1.27)) (justify left))
-  )
-  (hierarchical_label "Flash" (shape input) (at 208.28 40.64 180)
-    (effects (font (size 1.27 1.27)) (justify right))
-  )
-  (hierarchical_label "TX" (shape bidirectional) (at 208.28 43.18 180)
-    (effects (font (size 1.27 1.27)) (justify right))
-  )
-  (hierarchical_label "RX" (shape bidirectional) (at 208.28 45.72 180)
-    (effects (font (size 1.27 1.27)) (justify right))
-  )
-  (hierarchical_label "Reset" (shape input) (at 247.65 43.18 0)
     (effects (font (size 1.27 1.27)) (justify left))
   )
@@
     (pin "1")
   )
+  (symbol (lib_id "power:+3V3") (at 129.54 74.295 0) (unit 1)
+    (in_bom yes) (on_board yes) (fields_autoplaced)
+    (property "Reference" "#PWR036" (id 0) (at 129.54 78.105 0)
+      (effects (font (size 1.27 1.27)) hide)
+    )
+    (property "Value" "+3V3" (id 1) (at 129.54 69.215 0))
+    (property "Footprint" "" (id 2) (at 129.54 74.295 0)
+      (effects (font (size 1.27 1.27)) hide)
+    )
+    (property "Datasheet" "" (id 3) (at 129.54 74.295 0)
+      (effects (font (size 1.27 1.27)) hide)
+    )
+    (pin "1")
+  )
   (symbol (lib_id "power:+3V3") (at 160.02 34.29 0) (unit 1)
     (in_bom yes) (on_board yes) (fields_autoplaced)
@@
     )
     (property "Datasheet" "" (id 3) (at 160.02 34.29 0)
-      (effects (font (size 1.27 1.27)) hide)
-    )
-    (pin "1")
-  )
-  (symbol (lib_id "power:+3V3") (at 243.84 34.29 0) (unit 1)
-    (in_bom yes) (on_board yes) (fields_autoplaced)
-    (property "Reference" "#PWR036" (id 0) (at 243.84 38.1 0)
-      (effects (font (size 1.27 1.27)) hide)
-    )
-    (property "Value" "+3V3" (id 1) (at 243.84 29.21 0))
-    (property "Footprint" "" (id 2) (at 243.84 34.29 0)
-      (effects (font (size 1.27 1.27)) hide)
-    )
-    (property "Datasheet" "" (id 3) (at 243.84 34.29 0)
       (effects (font (size 1.27 1.27)) hide)
     )
@@
     (pin "1")
   )
+  (symbol (lib_id "power:GND") (at 130.81 92.075 0) (unit 1)
+    (in_bom yes) (on_board yes) (fields_autoplaced)
+    (property "Reference" "#PWR037" (id 0) (at 130.81 98.425 0)
+      (effects (font (size 1.27 1.27)) hide)
+    )
+    (property "Value" "GND" (id 1) (at 130.81 97.155 0))
+    (property "Footprint" "" (id 2) (at 130.81 92.075 0)
+      (effects (font (size 1.27 1.27)) hide)
+    )
+    (property "Datasheet" "" (id 3) (at 130.81 92.075 0)
+      (effects (font (size 1.27 1.27)) hide)
+    )
+    (pin "1")
+  )
   (symbol (lib_id "power:GND") (at 160.02 113.03 0) (unit 1)
     (in_bom yes) (on_board yes) (fields_autoplaced)
@@
     )
     (property "Datasheet" "" (id 3) (at 160.02 113.03 0)
-      (effects (font (size 1.27 1.27)) hide)
-    )
-    (pin "1")
-  )
-  (symbol (lib_id "power:GND") (at 245.11 52.07 0) (unit 1)
-    (in_bom yes) (on_board yes) (fields_autoplaced)
-    (property "Reference" "#PWR037" (id 0) (at 245.11 58.42 0)
-      (effects (font (size 1.27 1.27)) hide)
-    )
-    (property "Value" "GND" (id 1) (at 245.11 57.15 0))
-    (property "Footprint" "" (id 2) (at 245.11 52.07 0)
-      (effects (font (size 1.27 1.27)) hide)
-    )
-    (property "Datasheet" "" (id 3) (at 245.11 52.07 0)
       (effects (font (size 1.27 1.27)) hide)
     )
@@
   )
   (symbol (lib_id "Device:Q_PMOS_SGD") (at 76.2 121.92 0) (unit 1)
-    (in_bom yes) (on_board yes) (fields_autoplaced)
+    (in_bom yes) (on_board yes)
     (property "Reference" "Q5" (id 0) (at 82.55 120.6499 0)
       (effects (font (size 1.27 1.27)) (justify left))
@@
     (pin "3")
   )
-  (symbol (lib_id "TC2030-IDC:TC2030-IDC") (at 226.06 43.18 0) (unit 1)
-    (in_bom yes) (on_board yes) (fields_autoplaced)
-    (property "Reference" "ESP1" (id 0) (at 227.33 33.02 0))
-    (property "Value" "ESP Programming TagConnect" (id 1) (at 227.33 35.56 0))
-    (property "Footprint" "TC2030-IDC:Tag-Connect_TC2030-IDC-NL_2x03_P1.27mm_Vertical" (id 2) (at 226.06 43.18 0)
-      (effects (font (size 1.27 1.27)) hide)
-    )
-    (property "Datasheet" "None" (id 3) (at 226.06 43.18 0)
+  (symbol (lib_id "TC2030-IDC:TC2030-IDC") (at 111.76 83.185 0) (unit 1)
+    (in_bom yes) (on_board yes) (fields_autoplaced)
+    (property "Reference" "ESP1" (id 0) (at 113.03 73.025 0))
+    (property "Value" "ESP Programming TagConnect" (id 1) (at 113.03 75.565 0))
+    (property "Footprint" "TC2030-IDC:Tag-Connect_TC2030-IDC-NL_2x03_P1.27mm_Vertical" (id 2) (at 111.76 83.185 0)
+      (effects (font (size 1.27 1.27)) hide)
+    )
+    (property "Datasheet" "None" (id 3) (at 111.76 83.185 0)
       (effects (font (size 1.27 1.27)) (justify left bottom) hide)
     )
-    (property "Field4" "Tag-Connect LLC" (id 4) (at 226.06 43.18 0)
+    (property "Field4" "Tag-Connect LLC" (id 4) (at 111.76 83.185 0)
       (effects (font (size 1.27 1.27)) (justify left bottom) hide)
     )
-    (property "Field5" "None" (id 5) (at 226.06 43.18 0)
+    (property "Field5" "None" (id 5) (at 111.76 83.185 0)
       (effects (font (size 1.27 1.27)) (justify left bottom) hide)
     )
-    (property "Field6" "TC2030-IDC" (id 6) (at 226.06 43.18 0)
+    (property "Field6" "TC2030-IDC" (id 6) (at 111.76 83.185 0)
       (effects (font (size 1.27 1.27)) (justify left bottom) hide)
     )
-    (property "Field7" "Cable Adapter 6 Pos" (id 7) (at 226.06 43.18 0)
+    (property "Field7" "Cable Adapter 6 Pos" (id 7) (at 111.76 83.185 0)
       (effects (font (size 1.27 1.27)) (justify left bottom) hide)
     )
