File: Electrical/Swarmbot/Motors.kicad_sch (KiCad schematic)
At the start: 8 parts, among them J6 Motor 1, J7 Motor 2, U10 MPC17531A

Commit message: some little changes have been made
Parts:
- removed J6: Motor 1, Connector_JST:JST_XH_B2B-XH-AM_1x02_P2.50mm_Vertical, symbol Connector_Generic:Conn_01x02
- removed J7: Motor 2, Connector_JST:JST_XH_B2B-XH-AM_1x02_P2.50mm_Vertical, symbol Connector_Generic:Conn_01x02
- added J6: Motors, Connector_JST:JST_XH_B4B-XH-AM_1x04_P2.50mm_Vertical, symbol Connector_Generic:Conn_01x04
Connections:
- net Motor 1A: now also J6.1 (Pin_1)
- net Motor 1B: now also J6.2 (Pin_2)
- net Motor 2A: now also J6.3 (Pin_3)
- net Motor 2B: now also J6.4 (Pin_4)
Changed lines of the file:
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@@
     (stroke (width 0) (type default) (color 0 0 0 0))
   )
-  (wire (pts (xy 126.365 83.185) (xy 135.255 83.185))
-    (stroke (width 0) (type default) (color 0 0 0 0))
-  )
-  (wire (pts (xy 126.365 85.725) (xy 135.255 85.725))
+  (wire (pts (xy 126.365 83.185) (xy 132.08 83.185))
+    (stroke (width 0) (type default) (color 0 0 0 0))
+  )
+  (wire (pts (xy 126.365 85.725) (xy 132.08 85.725))
     (stroke (width 0) (type default) (color 0 0 0 0))
   )
@@
   )
   (wire (pts (xy 128.905 109.855) (xy 137.16 109.855))
+    (stroke (width 0) (type default) (color 0 0 0 0))
+  )
+  (wire (pts (xy 132.08 81.915) (xy 132.08 83.185))
+    (stroke (width 0) (type default) (color 0 0 0 0))
+  )
+  (wire (pts (xy 132.08 84.455) (xy 132.08 85.725))
+    (stroke (width 0) (type default) (color 0 0 0 0))
+  )
+  (wire (pts (xy 135.255 81.915) (xy 132.08 81.915))
+    (stroke (width 0) (type default) (color 0 0 0 0))
+  )
+  (wire (pts (xy 135.255 84.455) (xy 132.08 84.455))
     (stroke (width 0) (type default) (color 0 0 0 0))
   )
@@
     (pin "2")
   )
-  (symbol (lib_id "Connector_Generic:Conn_01x02") (at 140.335 79.375 0) (mirror x) (unit 1)
-    (in_bom yes) (on_board yes)
-    (property "Reference" "J6" (id 0) (at 142.367 79.1718 0)
-      (effects (font (size 1.27 1.27)) (justify left))
-    )
-    (property "Value" "Motor 1" (id 1) (at 142.367 76.8604 0)
-      (effects (font (size 1.27 1.27)) (justify left))
-    )
-    (property "Footprint" "Connector_JST:JST_XH_B2B-XH-AM_1x02_P2.50mm_Vertical" (id 2) (at 140.335 79.375 0)
+  (symbol (lib_id "Connector_Generic:Conn_01x04") (at 140.335 79.375 0) (unit 1)
+    (in_bom yes) (on_board yes)
+    (property "Reference" "J6" (id 0) (at 142.367 79.5782 0)
+      (effects (font (size 1.27 1.27)) (justify left))
+    )
+    (property "Value" "Motors" (id 1) (at 142.367 81.8896 0)
+      (effects (font (size 1.27 1.27)) (justify left))
+    )
+    (property "Footprint" "Connector_JST:JST_XH_B4B-XH-AM_1x04_P2.50mm_Vertical" (id 2) (at 140.335 79.375 0)
       (effects (font (size 1.27 1.27)) hide)
     )
@@
     (pin "1")
     (pin "2")
-  )
-  (symbol (lib_id "Connector_Generic:Conn_01x02") (at 140.335 85.725 0) (mirror x) (unit 1)
-    (in_bom yes) (on_board yes)
-    (property "Reference" "J7" (id 0) (at 142.367 85.5218 0)
-      (effects (font (size 1.27 1.27)) (justify left))
-    )
-    (property "Value" "Motor 2" (id 1) (at 142.367 83.2104 0)
-      (effects (font (size 1.27 1.27)) (justify left))
-    )
-    (property "Footprint" "Connector_JST:JST_XH_B2B-XH-AM_1x02_P2.50mm_Vertical" (id 2) (at 140.335 85.725 0)
-      (effects (font (size 1.27 1.27)) hide)
-    )
-    (property "Datasheet" "~" (id 3) (at 140.335 85.725 0)
-      (effects (font (size 1.27 1.27)) hide)
-    )
-    (pin "1")
-    (pin "2")
+    (pin "3")
+    (pin "4")
   )
   (symbol (lib_id "MPC17531ATEJ - H Bridge:MPC17531A") (at 111.125 90.805 0) (unit 1)

Commit message: some little changes have been made
Parts:
- J6: footprint Connector_JST:JST_XH_B4B-XH-AM_1x04_P2.50mm_Vertical -> Connector_JST:JST_XH_B4B-XH-A_1x04_P2.50mm_Vertical
Changed lines of the file:
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@@
       (effects (font (size 1.27 1.27)) (justify left))
     )
-    (property "Footprint" "Connector_JST:JST_XH_B4B-XH-AM_1x04_P2.50mm_Vertical" (id 2) (at 140.335 79.375 0)
+    (property "Footprint" "Connector_JST:JST_XH_B4B-XH-A_1x04_P2.50mm_Vertical" (id 2) (at 140.335 79.375 0)
       (effects (font (size 1.27 1.27)) hide)
     )

Commit message: off to do other things for a second
;
Parts:
- added J7: Sensors, Connector_JST:JST_XH_B4B-XH-A_1x04_P2.50mm_Vertical, symbol Connector_Generic:Conn_01x04
Connections:
- net +3V3: now also J7.1 (Pin_1)
- net GND: now also J7.4 (Pin_4)
- new net Motor Sensor 1: J7.2 (Pin_2)
- new net Motor Sensor 2: J7.3 (Pin_3)
Changed lines of the file:
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@@
+    (stroke (width 0) (type default) (color 0 0 0 0))
+  )
+  (wire (pts (xy 201.295 80.645) (xy 213.36 80.645))
+    (stroke (width 0) (type default) (color 0 0 0 0))
+  )
+  (wire (pts (xy 201.295 83.185) (xy 213.36 83.185))
+    (stroke (width 0) (type default) (color 0 0 0 0))
+  )
+  (wire (pts (xy 211.455 78.105) (xy 211.455 74.295))
+    (stroke (width 0) (type default) (color 0 0 0 0))
+  )
+  (wire (pts (xy 211.455 85.725) (xy 211.455 88.9))
+    (stroke (width 0) (type default) (color 0 0 0 0))
+  )
+  (wire (pts (xy 213.36 78.105) (xy 211.455 78.105))
+    (stroke (width 0) (type default) (color 0 0 0 0))
+  )
+  (wire (pts (xy 213.36 85.725) (xy 211.455 85.725))
     (stroke (width 0) (type default) (color 0 0 0 0))
   )
@@
     (effects (font (size 1.27 1.27)) (justify right))
   )
+  (hierarchical_label "Motor Sensor 1" (shape output) (at 201.295 80.645 180)
+    (effects (font (size 1.27 1.27)) (justify right))
+  )
+  (hierarchical_label "Motor Sensor 2" (shape output) (at 201.295 83.185 180)
+    (effects (font (size 1.27 1.27)) (justify right))
+  )
   (symbol (lib_id "power:+BATT") (at 76.2 115.57 0) (unit 1)
     (in_bom yes) (on_board yes)
@@
     (pin "1")
   )
+  (symbol (lib_id "power:+3V3") (at 211.455 74.295 0) (unit 1)
+    (in_bom yes) (on_board yes) (fields_autoplaced)
+    (property "Reference" "#PWR0118" (id 0) (at 211.455 78.105 0)
+      (effects (font (size 1.27 1.27)) hide)
+    )
+    (property "Value" "+3V3" (id 1) (at 211.455 69.215 0))
+    (property "Footprint" "" (id 2) (at 211.455 74.295 0)
+      (effects (font (size 1.27 1.27)) hide)
+    )
+    (property "Datasheet" "" (id 3) (at 211.455 74.295 0)
+      (effects (font (size 1.27 1.27)) hide)
+    )
+    (pin "1")
+  )
   (symbol (lib_id "power:GND") (at 76.2 125.73 0) (unit 1)
     (in_bom yes) (on_board yes) (fields_autoplaced)
@@
     (pin "1")
   )
+  (symbol (lib_id "power:GND") (at 211.455 88.9 0) (unit 1)
+    (in_bom yes) (on_board yes) (fields_autoplaced)
+    (property "Reference" "#PWR0117" (id 0) (at 211.455 95.25 0)
+      (effects (font (size 1.27 1.27)) hide)
+    )
+    (property "Value" "GND" (id 1) (at 211.455 93.98 0))
+    (property "Footprint" "" (id 2) (at 211.455 88.9 0)
+      (effects (font (size 1.27 1.27)) hide)
+    )
+    (property "Datasheet" "" (id 3) (at 211.455 88.9 0)
+      (effects (font (size 1.27 1.27)) hide)
+    )
+    (pin "1")
+  )
   (symbol (lib_id "Device:C_Small") (at 76.2 121.285 0) (unit 1)
     (in_bom yes) (on_board yes) (fields_autoplaced)
@@
       (effects (font (size 1.27 1.27)) hide)
     )
+    (pin "1")
+    (pin "2")
+    (pin "3")
+    (pin "4")
+  )
+  (symbol (lib_id "Connector_Generic:Conn_01x04") (at 218.44 80.645 0) (unit 1)
+    (in_bom yes) (on_board yes)
+    (property "Reference" "J7" (id 0) (at 220.472 80.8482 0)
+      (effects (font (size 1.27 1.27)) (justify left))
+    )
+    (property "Value" "Sensors" (id 1) (at 220.472 83.1596 0)
+      (effects (font (size 1.27 1.27)) (justify left))
+    )
+    (property "Footprint" "Connector_JST:JST_XH_B4B-XH-A_1x04_P2.50mm_Vertical" (id 2) (at 218.44 80.645 0)
+      (effects (font (size 1.27 1.27)) hide)
+    )
+    (property "Datasheet" "~" (id 3) (at 218.44 80.645 0)
+      (effects (font (size 1.27 1.27)) hide)
+    )

Commit message: Made some Changes
Parts:
- removed J6: Motors, Connector_JST:JST_XH_B4B-XH-A_1x04_P2.50mm_Vertical, symbol Connector_Generic:Conn_01x04
- removed J7: Sensors, Connector_JST:JST_XH_B4B-XH-A_1x04_P2.50mm_Vertical, symbol Connector_Generic:Conn_01x04
- renumbered C23 to C4, C24 to C5, C20 to C6, C21 to C7, C22 to C8, U10 to U6
Connections:
- net +3V3 renamed Motor 3V3
- net +BATT renamed Motor 5V
- net GND renamed Motor GND
- net Motor 1A renamed H-Bridge 1A
- net Motor 1B renamed H-Bridge 1B
- net Motor 2A renamed H-Bridge 2A
- net Motor 2B renamed H-Bridge 2B

Commit message: some pcb changes
Parts:
- added C27: 100pF, Capacitor_SMD:C_0805_2012Metric_Pad1.18x1.45mm_HandSolder, symbol Device:C_Small
Connections:
- net Motor 5V: now also C27.1
- net Motor GND: now also C27.2
Changed lines of the file:
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@@
   (junction (at 76.2 113.03) (diameter 0) (color 0 0 0 0))
   (junction (at 76.2 129.54) (diameter 0) (color 0 0 0 0))
+  (junction (at 86.995 113.03) (diameter 0) (color 0 0 0 0))
   (junction (at 86.995 129.54) (diameter 0) (color 0 0 0 0))
+  (junction (at 97.155 129.54) (diameter 0) (color 0 0 0 0))
   (junction (at 111.125 119.38) (diameter 0) (color 0 0 0 0))
   (junction (at 111.125 129.54) (diameter 0) (color 0 0 0 0))
@@
     (stroke (width 0) (type default) (color 0 0 0 0))
   )
-  (wire (pts (xy 86.995 129.54) (xy 111.125 129.54))
+  (wire (pts (xy 86.995 129.54) (xy 97.155 129.54))
     (stroke (width 0) (type default) (color 0 0 0 0))
   )
@@
   )
   (wire (pts (xy 93.98 85.725) (xy 98.425 85.725))
+    (stroke (width 0) (type default) (color 0 0 0 0))
+  )
+  (wire (pts (xy 97.155 113.03) (xy 86.995 113.03))
+    (stroke (width 0) (type default) (color 0 0 0 0))
+  )
+  (wire (pts (xy 97.155 118.745) (xy 97.155 113.03))
+    (stroke (width 0) (type default) (color 0 0 0 0))
+  )
+  (wire (pts (xy 97.155 123.825) (xy 97.155 129.54))
+    (stroke (width 0) (type default) (color 0 0 0 0))
+  )
+  (wire (pts (xy 97.155 129.54) (xy 111.125 129.54))
     (stroke (width 0) (type default) (color 0 0 0 0))
   )
@@
       (effects (font (size 1.27 1.27)) hide)
     )
+    (pin "1")
+    (pin "2")
+  )
+  (symbol (lib_id "Device:C_Small") (at 97.155 121.285 0) (unit 1)
+    (in_bom yes) (on_board yes) (fields_autoplaced)
+    (property "Reference" "C27" (id 0) (at 99.695 120.0149 0)
+      (effects (font (size 1.27 1.27)) (justify left))
+    )
+    (property "Value" "100pF" (id 1) (at 99.695 122.5549 0)
+      (effects (font (size 1.27 1.27)) (justify left))
+    )
+    (property "Footprint" "Capacitor_SMD:C_0805_2012Metric_Pad1.18x1.45mm_HandSolder" (id 2) (at 97.155 121.285 0)
+      (effects (font (size 1.27 1.27)) hide)
+    )
+    (property "Datasheet" "~" (id 3) (at 97.155 121.285 0)
+      (effects (font (size 1.27 1.27)) hide)
+    )
