File: Electrical/Swarmbot/swarmbot.kicad_pcb (KiCad board)
At the start: 4 copper layers, 100 x 80 mm, 92 parts, among them J1 Conn_02x07_Counter_Clockwise, J2 Conn_02x07_Counter_Clockwise, J3 Charging Header, J4 Battery 1S2P, J5 Raspberry_Pi_2_3, J6 Motor 1, J7 Motor 2, Q1 BSH108, Q2 BSH108, Q3 BSH108, Q4 BSH108, Q5 RSC002P03, Q6 RSC002P03, SW1 Left, SW2 Right, SW3 SW_SPST, U1 QRE1113GR, U10 MPC17531A, U2 QRE1113GR, U3 QRE1113GR, U4 QRE1113GR, U5 ESP32-WROOM-32D, U6 TP4056, U8 AP9101CK, U9 AP2112K-3.3

Commit message: some little changes have been made
Parts:
- removed J7: Motor 2, Connector_JST:JST_XH_B2B-XH-AM_1x02_P2.50mm_Vertical
- added C25: 100pF, Capacitor_SMD:C_0805_2012Metric_Pad1.18x1.45mm_HandSolder, F.Cu at (239.9, 105.4)
- added C26: 100nF, Capacitor_SMD:C_0805_2012Metric_Pad1.18x1.45mm_HandSolder, B.Cu at (144.1, 117.6)
- added R31: .0025R, Resistor_SMD:R_1206_3216Metric_Pad1.30x1.75mm_HandSolder, B.Cu at (139.8, 121.4)
- added R32: 2k7, Resistor_SMD:R_0805_2012Metric_Pad1.20x1.40mm_HandSolder, B.Cu at (144.1, 115.4)
- added R33: 470, Resistor_SMD:R_0805_2012Metric_Pad1.20x1.40mm_HandSolder, B.Cu at (206.6, 121.3)
- added R34: 10k, Resistor_SMD:R_0805_2012Metric_Pad1.20x1.40mm_HandSolder, B.Cu at (200.9, 128.7)
- added Servo1: Conn_01x03_Male, Connector_PinHeader_2.54mm:PinHeader_1x03_P2.54mm_Vertical, B.Cu at (143.8, 86.4)
- added Sonar1: Conn_01x04_Male, Connector_PinHeader_2.54mm:PinHeader_1x04_P2.54mm_Vertical, F.Cu at (208.8, 96.3)
- added U11: INA138, Package_TO_SOT_SMD:SOT-23-5, B.Cu at (139.8, 117.0)
- added U12: QRE1113GR, OptoDevice:OnSemi_CASE100CY, B.Cu at (206.6, 126.6)
- J6: value Motor 1 -> Motors; footprint Connector_JST:JST_XH_B2B-XH-AM_1x02_P2.50mm_Vertical -> Connector_JST:JST_XH_B4B-XH-AM_1x04_P2.50mm_Vertical
- Logo2: moved to F.Cu
- R18, R19, R23: moved to B.Cu
- moved R27 131.7 mm to (94.1, 48.9)
- moved R26 130.6 mm to (93.7, 53.4)
- moved R25 129.9 mm to (90.9, 56.4)
- moved R22 129.1 mm to (86.2, 56.4)
- moved C4 129.0 mm to (104.6, 51.9)
- moved C14 127.2 mm to (81.4, 55.1)
- moved C15 125.4 mm to (76.3, 59.5)
- moved C13 122.1 mm to (89.0, 53.4)
- moved C8 119.9 mm to (81.1, 59.5)
- moved C3 111.9 mm to (104.6, 48.9)
- moved U6 110.4 mm to (80.2, 50.5)
- moved U8 110.4 mm to (89.1, 49.7)
- moved R24 106.4 mm to (85.9, 59.3)
- moved U9 96.9 mm to (76.4, 55.8)
- moved R2 70.5 mm to (258.8, 99.0), turned to 0 degrees
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Connections:
- net /Charging Pad Top renamed /Line Sensor 5 Top
- net Net-(J4-Pad1) renamed /Top PCB/Power/Bat+VE
- D2 pad 2: /Top PCB/Power/PowerIn -> /Charging Top Pad
- D7 pad 2: /Top PCB/Power/PowerIn -> /Charging Top Pad
- J1 pad 11: unconnected-(J1-Pad11) -> /Sonar Echo Top
- J1 pad 12: unconnected-(J1-Pad12) -> /Sonar Trigger Top
- J1 pad 3: GND -> +5V
- J2 pad 11: unconnected-(J2-Pad11) -> /Sonar Echo Lower
- J2 pad 12: unconnected-(J2-Pad12) -> /Sonar Trigger Lower
- J2 pad 3: GND -> /Sonar 5V Lower
- J2 pad 7: /Charging Pad Lower -> /Line Sensor 5 Lower
- J3 pad 1: /Top PCB/Power/PowerIn -> /Charging Top Pad
- J6 pad 1: /Top PCB/Motors/Motor 1B -> /Top PCB/Motors/Motor 1A
- J6 pad 2: /Top PCB/Motors/Motor 1A -> /Top PCB/Motors/Motor 1B
- U5 pad 11: /Top PCB/ESP32/Motor Sensor 1 -> /Sonar Trigger Top
- U5 pad 12: /Top PCB/ESP32/Motor Sensor 2 -> /Sonar Echo Top
- U5 pad 13: /Left Switch Top -> /Right Switch Top
- U5 pad 14: /Right Switch Top -> /Left Switch Top
- U5 pad 33: /Top PCB/ESP32/Sonar Echo -> /Top PCB/ESP32/Motor Sensor 1
- U5 pad 36: /Top PCB/ESP32/Sonar Trigger -> /Top PCB/ESP32/Motor Sensor 2
Routing:
- net /Top PCB/ESP32/Bat I: track 0.00 -> 56.9 mm, vias 0 -> 2
- net +5V: track 53.8 -> 109.8 mm, vias 0 -> 1
- net /Sonar 5V Lower: track 0.00 -> 42.5 mm
- net /Charging Top Pad: track 0.00 -> 42.2 mm
- net +BATT: track 81.9 -> 123.4 mm
- net /Right Switch Lower: track 36.8 -> 0.00 mm
- net /Line Sensor 2 Lower: track 34.3 -> 2.94 mm
- net /Line Sensor 1 Lower: track 35.0 -> 4.25 mm
- net /Sonar Trigger Top: track 0.00 -> 29.0 mm
- net /Top PCB/Power/PowerInInrush: track 0.00 -> 28.7 mm, vias 0 -> 2
- net /Line Sensor 3 Lower: track 30.6 -> 2.69 mm
- net /Sonar Echo Top: track 0.00 -> 26.5 mm
- net GND: track 81.4 -> 107.2 mm, vias 54 -> 50
- net /Sonar Trigger Lower: track 0.00 -> 25.4 mm
- net /Line Sensor 4 Lower: track 29.7 -> 4.83 mm
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
Commit message: some little changes have been made
Parts:
- C18, C19, C25, R1, R2: moved to B.Cu
- J6: footprint Connector_JST:JST_XH_B4B-XH-AM_1x04_P2.50mm_Vertical -> Connector_JST:JST_XH_B4B-XH-A_1x04_P2.50mm_Vertical
- Sonar1: footprint Connector_PinHeader_2.54mm:PinHeader_1x04_P2.54mm_Vertical -> Connector_PinSocket_2.54mm:PinSocket_1x04_P2.54mm_Vertical
- moved R2 66.4 mm to (195.8, 120.1), turned to 180 degrees
- moved C18 63.2 mm to (188.3, 114.9), turned to 180 degrees
- moved R1 57.7 mm to (195.6, 79.9), turned to 180 degrees
- moved C19 47.1 mm to (188.3, 111.4), turned to 180 degrees
- moved C25 32.9 mm to (209.7, 92.3)
Routing:
- net /Right Switch Lower: track 0.00 -> 39.7 mm
- net /Line Sensor 3 Lower: track 2.69 -> 41.3 mm
- net /Line Sensor 1 Lower: track 4.25 -> 36.1 mm
- net /Sonar Echo Lower: track 7.94 -> 39.1 mm
- net /Line Sensor 2 Lower: track 2.94 -> 33.8 mm
- net /Line Sensor LEDs Lower: track 72.1 -> 98.2 mm
- net /Line Sensor 4 Lower: track 4.83 -> 30.2 mm
- net /Line Sensor 5 Lower: track 17.9 -> 38.8 mm
- net GND: track 107.2 -> 127.8 mm, vias 50 -> 53
- net /Left Switch Lower: track 0.00 -> 20.2 mm
- net /Sonar Trigger Lower: track 25.4 -> 34.1 mm
- net /Sonar 5V Lower: track 42.5 -> 46.0 mm
- net /Top PCB/Motors/Motor 1B: track 24.8 -> 23.7 mm
- net /Charging Pad Lower: track 40.1 -> 39.6 mm
Other:
- board text added: "+5 VDC"
- board text added: "Swarmbot Version 0.1"

Commit message: off to do other things for a second
;
Parts:
- added J7: Sensors, Connector_JST:JST_XH_B4B-XH-A_1x04_P2.50mm_Vertical, B.Cu at (139.3, 86.1)
- moved Servo1 9.50 mm to (136.3, 80.5), turned to -90 degrees
Routing:
- net +5V: track 109.8 -> 116.1 mm
- net /Top PCB/ESP32/Pen Servo: track 7.40 -> 9.50 mm
Other:
- board text added: "Don't Panic!"
- board text added: "Swarmbot Version 0.2"
- board text added: "Version 0.2"
- board text removed: "Don't ask!"
- board text removed: "Version 0.1"

Commit message: Made some Changes
Parts:
- removed J6: Motors, Connector_JST:JST_XH_B4B-XH-A_1x04_P2.50mm_Vertical
- removed J7: Sensors, Connector_JST:JST_XH_B4B-XH-A_1x04_P2.50mm_Vertical
- added R35: 470, Resistor_SMD:R_0805_2012Metric_Pad1.20x1.40mm_HandSolder, F.Cu at (202.0, 38.1)
- added R36: 470, Resistor_SMD:R_0805_2012Metric_Pad1.20x1.40mm_HandSolder, F.Cu at (206.8, 41.0)
- added R37: 10k, Resistor_SMD:R_0805_2012Metric_Pad1.20x1.40mm_HandSolder, F.Cu at (206.8, 38.1)
- added R38: 10k, Resistor_SMD:R_0805_2012Metric_Pad1.20x1.40mm_HandSolder, F.Cu at (202.0, 41.0)
- added U7: ESP32-WROOM-32D, RF_Module:ESP32-WROOM-32, F.Cu at (112.6, 125.8)
- C1, C2, C9, D1, D2, D6, D7, H1, H2, J4, J5, L1, Q1, Q2, Q3, Q4, Q5, Q6, R1, R10, R11, R12, R13, R14, R15, R16, R2, R3, R30, R4, R5, R6, R8, R9, SW3, Servo1, U1, U2, U3, U4: moved to F.Cu
- C10: value 100nF -> 10uF; moved to F.Cu
- C11: value 22uF -> 10uF; moved to F.Cu
- C12, C7: value 22uF -> 100pF; moved to F.Cu
- C13: value 1uF -> 10uF
- C15: value 1uF -> 22uF
- C16, C19: value 10uF -> 22uF; moved to F.Cu
- C17, C22, C25: value 100pF -> 10uF; moved to F.Cu
- C18: value 10uF -> 100nF; moved to F.Cu
- C20: value 100pF -> 22uF; moved to F.Cu
- C21, C23: value 100pF -> 1uF; moved to F.Cu
- C24: value 100pF -> 100nF; moved to F.Cu
- C26: value 100nF -> 100pF; moved to F.Cu
- C3: value 10uF -> 100pF
- C5, C6: value 10uF -> 100pF; moved to F.Cu
- C8: value 22uF -> 100pF
- ESP1, J3: moved to B.Cu
- J1: value Conn_02x07_Counter_Clockwise -> 12x2 JST; footprint Connector_JST:JST_PUD_B14B-PUDSS_2x07_P2.00mm_Vertical -> Connector_JST:JST_PUD_B24B-PUDSS_2x12_P2.00mm_Vertical; moved to F.Cu
- J2: value Conn_02x07_Counter_Clockwise -> 12x2 JST; footprint Connector_JST:JST_PUD_B14B-PUDSS_2x07_P2.00mm_Vertical -> Connector_JST:JST_PUD_B24B-PUDSS_2x12_P2.00mm_Vertical
- Logo2: footprint SquashedFly Logo:SquashedFlyBrightCopper -> SquashedFly Logo:SquashedFlySilk
- R17, R20, R21: value 1k -> 10k
- R18, R19: value 2R -> 10k; moved to F.Cu
- R22: value 30k -> 1k
- R23: value 1k2 -> 2R; moved to F.Cu
- R24: value 73k -> 2R
- R25: value 10k -> 1k
- R26: value 2k7 -> 1k
- R27: value 330 -> 30k
- R28: value 10k -> 1k2; moved to F.Cu
- R29: value 10k -> 73k; moved to F.Cu
- R31: value .0025R -> 2k7; footprint Resistor_SMD:R_1206_3216Metric_Pad1.30x1.75mm_HandSolder -> Resistor_SMD:R_0805_2012Metric_Pad1.20x1.40mm_HandSolder; moved to F.Cu
- R32: value 2k7 -> 330; moved to F.Cu
- R33: value 470 -> .0025R; footprint Resistor_SMD:R_0805_2012Metric_Pad1.20x1.40mm_HandSolder -> Resistor_SMD:R_1206_3216Metric_Pad1.30x1.75mm_HandSolder; moved to F.Cu
- R34: value 10k -> 2k7; moved to F.Cu
- R7: value 10k -> 470; moved to F.Cu
- U10: value MPC17531A -> AP9101CK; footprint Package_SO:HTSSOP-20-1EP_4.4x6.5mm_P0.65mm_EP3.4x6.5mm_Mask2.75x3.43mm_ThermalVias_HandSolder -> Package_TO_SOT_SMD:SOT-23-5; moved to F.Cu
- U11: value INA138 -> AP2112K-3.3; moved to F.Cu
- U12: value QRE1113GR -> INA138; footprint OptoDevice:OnSemi_CASE100CY -> Package_TO_SOT_SMD:SOT-23-5; moved to F.Cu
- U5: value ESP32-WROOM-32D -> QRE1113GR; footprint RF_Module:ESP32-WROOM-32 -> OptoDevice:OnSemi_CASE100CY; moved to F.Cu
- U6: value TP4056 -> MPC17531A; footprint Package_SO:SOP-8-1EP_4.57x4.57mm_P1.27mm_EP4.57x4.45mm_ThermalVias -> Package_SO:HTSSOP-20-1EP_4.4x6.5mm_P0.65mm_EP3.4x6.5mm_Mask2.75x3.43mm_ThermalVias_HandSolder
- U8: value AP9101CK -> TP4056; footprint Package_TO_SOT_SMD:SOT-23-5 -> Package_SO:SOP-8-1EP_4.57x4.57mm_P1.27mm_EP4.57x4.45mm_ThermalVias
- moved U4 212.7 mm to (14.2, 41.6), turned to 0 degrees
- moved U3 206.9 mm to (19.0, 41.6), turned to 0 degrees
- moved C25 200.6 mm to (14.3, 46.7)
- moved U1 199.7 mm to (9.47, 41.6), turned to 0 degrees
- moved U12 196.2 mm to (33.0, 35.2), turned to 0 degrees
- moved R34 195.7 mm to (23.8, 45.4)
- moved R33 195.6 mm to (28.5, 40.3)
- moved R4 192.3 mm to (23.8, 48.4)
- moved R29 191.0 mm to (37.7, 25.9)
- moved R30 190.8 mm to (37.7, 28.8)
- moved U2 190.5 mm to (33.0, 28.0), turned to 0 degrees
- moved C19 190.2 mm to (9.51, 46.7), turned to 0 degrees
- moved R5 189.4 mm to (37.7, 34.7)
- moved R6 189.3 mm to (42.5, 28.8)
- moved H2 188.2 mm to (42.1, 32.3), turned to 0 degrees
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Connections:
- C1 pad 1: /Top PCB/ESP32/5V Switched 1 -> /Lower PCB 3V3
- C1 pad 2: GND -> /Lower PCB GND
- C10 pad 1: +BATT -> /Line Sensor LEDs Top
- C11 pad 1: +5V -> +3V3
- C12 pad 1: +5V -> +3V3
- C13 pad 1: /Top PCB/Power/VBAT -> /Top PCB/ESP32/Bat V
- C14 pad 1: +3V3 -> /Top PCB/Power/PowerInDiode
- C15 pad 1: +3V3 -> /Top PCB/Power/VBAT
- C16 pad 1: /Top PCB/ESP32/5V Switched 1 -> /Top PCB/Power/VBAT
- C17 pad 1: /Top PCB/ESP32/5V Switched 1 -> +BATT
- C18 pad 1: +3V3 -> +BATT
- C19 pad 1: +3V3 -> +5V
- C2 pad 1: /Line Sensor LEDs Top -> /Lower PCB 3V3
- C2 pad 2: GND -> /Lower PCB GND
- C20 pad 1: Net-(C20-Pad1) -> +5V
- C21 pad 1: Net-(C21-Pad1) -> /Top PCB/Power/VBAT
- C21 pad 2: Net-(C21-Pad2) -> GND
- C22 pad 1: Net-(C22-Pad1) -> +3V3
- C22 pad 2: Net-(C22-Pad2) -> GND
- C23 pad 1: +BATT -> +3V3
- C24 pad 1: +BATT -> /Top PCB/ESP32/Bat I
- C25 pad 1: /Sonar 5V Lower -> /Top PCB/ESP32/5V Switched 1
- C26 pad 1: /Top PCB/ESP32/Bat I -> /Top PCB/ESP32/5V Switched 1
- C3 pad 1: +3V3 -> /Lower PCB 5V
- C3 pad 2: GND -> /Lower PCB GND
- C4 pad 1: +3V3 -> /Lower PCB 5V
- C4 pad 2: GND -> /Lower PCB GND
- C5 pad 1: /Top PCB/ESP32/Bat V -> /Lower PCB 5V
- C5 pad 2: GND -> /Lower PCB GND
- C6 pad 1: /Top PCB/Power/PowerInDiode -> Net-(C6-Pad1)
- C6 pad 2: GND -> /Lower PCB GND
- C7 pad 1: /Top PCB/Power/VBAT -> Net-(C7-Pad1)
- C7 pad 2: GND -> Net-(C7-Pad2)
- C8 pad 1: /Top PCB/Power/VBAT -> Net-(C8-Pad1)
- C8 pad 2: GND -> Net-(C8-Pad2)
- C9 pad 1: +BATT -> /Top PCB/ESP32/5V Switched 1
- H2 pad 1: GND -> /Lower PCB GND
- J1 pad 10: /Line Sensor 1 Top -> GND
- J1 pad 11: /Sonar Echo Top -> /Line Sensor 3 Top
- J1 pad 12: /Sonar Trigger Top -> unconnected-(J1-Pad12)
- J1 pad 13: /Right Switch Top -> /Motor Sensor 1 Top
- J1 pad 14: /Left Switch Top -> /Motor Sensor 2 Top
- J1 pad 2: /Line Sensor LEDs Top -> +5V
- J1 pad 3: +5V -> GND
- J1 pad 4: /Line Sensor 4 Top -> /Charging Top Pad
- J1 pad 5: GND -> /H-Bridge 1B Top
- J1 pad 6: /Line Sensor 3 Top -> /H-Bridge 2B Top
- J1 pad 7: /Line Sensor 5 Top -> /H-Bridge 2A Top
- J1 pad 8: /Line Sensor 2 Top -> /H-Bridge 1A Top
- J1 pad 9: /Charging Top Pad -> GND
- J2 pad 1: +3V3 -> /Lower PCB 3V3
- J2 pad 10: /Line Sensor 1 Lower -> /Lower PCB GND
- J2 pad 11: /Sonar Echo Lower -> /Line Sensor 3 Lower
- J2 pad 12: /Sonar Trigger Lower -> unconnected-(J2-Pad12)
- J2 pad 13: /Right Switch Lower -> /Motor Sensor 1 Lower
- J2 pad 14: /Left Switch Lower -> /Motor Sensor 2 Lower
- J2 pad 2: /Line Sensor LEDs Lower -> /Lower PCB 5V
- J2 pad 3: /Sonar 5V Lower -> /Lower PCB GND
- J2 pad 4: /Line Sensor 4 Lower -> /Charging Pad Lower
- J2 pad 5: GND -> /H-Bridge 1B Lower
- J2 pad 6: /Line Sensor 3 Lower -> /H-Bridge 2B Lower
- J2 pad 7: /Line Sensor 5 Lower -> /H-Bridge 2A Lower
- J2 pad 8: /Line Sensor 2 Lower -> /H-Bridge 1A Lower
- J2 pad 9: /Charging Pad Lower -> /Lower PCB GND
- R1 pad 2: GND -> /Lower PCB GND
- R10 pad 1: /Top PCB/ESP32/Line Sensor LED -> /Lower PCB 3V3
- R10 pad 2: Net-(Q4-Pad1) -> /Line Sensor 3 Lower
- R11 pad 1: +3V3 -> /Lower PCB 3V3
- R11 pad 2: /Top PCB/ESP32/program -> /Line Sensor 4 Lower
- R12 pad 1: +3V3 -> /Lower PCB 3V3
- R12 pad 2: /Top PCB/ESP32/enable -> /Line Sensor 5 Lower
- R13 pad 1: +5V -> /Top PCB/ESP32/5V Switch Aux
- R13 pad 2: Net-(Q3-Pad3) -> Net-(Q3-Pad1)
- R14 pad 1: +5V -> /Top PCB/ESP32/5V Switch 1
- R14 pad 2: Net-(Q4-Pad3) -> Net-(Q3-Pad1)
- R15 pad 1: /Top PCB/ESP32/Bat V -> /Top PCB/ESP32/Line Sensor LED
- R15 pad 2: +BATT -> Net-(Q4-Pad1)
- R16 pad 1: GND -> +3V3
- R16 pad 2: /Top PCB/ESP32/Bat V -> /Top PCB/ESP32/program
- R17 pad 1: GND -> +3V3
- R17 pad 2: Net-(D3-Pad1) -> /Top PCB/ESP32/enable
- R18 pad 1: /Top PCB/Power/PowerInInrush -> +5V
- R18 pad 2: /Top PCB/Power/PowerInDiode -> Net-(Q3-Pad3)
- R19 pad 1: /Top PCB/Power/PowerInInrush -> +5V
- R19 pad 2: /Top PCB/Power/PowerInDiode -> Net-(Q4-Pad3)
- R2 pad 2: GND -> /Lower PCB GND
- R20 pad 1: Net-(R20-Pad1) -> /Top PCB/ESP32/Bat V
- R20 pad 2: Net-(D4-Pad1) -> +BATT
- R21 pad 1: Net-(D5-Pad1) -> GND
- R21 pad 2: Net-(R21-Pad2) -> /Top PCB/ESP32/Bat V
- R22 pad 2: Net-(R22-Pad2) -> Net-(D3-Pad1)
- R23 pad 1: GND -> /Top PCB/Power/PowerInInrush
- R23 pad 2: Net-(R23-Pad2) -> /Top PCB/Power/PowerInDiode
- R24 pad 1: Net-(R24-Pad1) -> /Top PCB/Power/PowerInInrush
- R24 pad 2: +5V -> /Top PCB/Power/PowerInDiode
- R25 pad 1: GND -> Net-(R25-Pad1)
- R25 pad 2: Net-(R24-Pad1) -> Net-(D4-Pad1)
- R26 pad 1: GND -> Net-(D5-Pad1)
- R27 pad 1: Net-(R27-Pad1) -> GND
- R27 pad 2: +BATT -> Net-(R27-Pad2)
- R28 pad 1: +3V3 -> GND
- R28 pad 2: /Line Sensor 2 Lower -> Net-(R28-Pad2)
- R29 pad 1: +3V3 -> Net-(R29-Pad1)
- R29 pad 2: /Line Sensor 3 Lower -> +5V
- R30 pad 1: +3V3 -> GND
- R30 pad 2: /Line Sensor 4 Lower -> Net-(R29-Pad1)
- R31 pad 1: /Top PCB/Power/Bat+VE -> GND
- R31 pad 2: +BATT -> Net-(R31-Pad2)
- R32 pad 1: /Top PCB/ESP32/Bat I -> Net-(R32-Pad1)
- R32 pad 2: Net-(R32-Pad2) -> +BATT
- R33 pad 1: /Line Sensor LEDs Lower -> /Top PCB/Power/Bat+VE
- R33 pad 2: Net-(R33-Pad2) -> +BATT
- R34 pad 1: +3V3 -> /Top PCB/ESP32/Bat I
- R34 pad 2: /Line Sensor 5 Lower -> Net-(R34-Pad2)
- R7 pad 1: +3V3 -> /Line Sensor LEDs Lower
- R7 pad 2: /Line Sensor 1 Lower -> Net-(R7-Pad2)
- R8 pad 1: /Top PCB/ESP32/5V Switch Aux -> /Lower PCB 3V3
- R8 pad 2: Net-(Q3-Pad1) -> /Line Sensor 1 Lower
- R9 pad 1: /Top PCB/ESP32/5V Switch 1 -> /Lower PCB 3V3
- R9 pad 2: Net-(Q3-Pad1) -> /Line Sensor 2 Lower
- SW1 pad 1: +3V3 -> /Lower PCB 3V3
- SW2 pad 1: +3V3 -> /Lower PCB 3V3
- Sonar1 pad 1: /Sonar 5V Lower -> /Lower PCB 5V
- Sonar1 pad 4: GND -> /Lower PCB GND
- U1 pad 2: GND -> /Lower PCB GND
- U1 pad 4: GND -> /Lower PCB GND
- U10 pad 1: +3V3 -> Net-(R31-Pad2)
- U10 pad 2: /Top PCB/ESP32/Motor PWM1 -> Net-(R32-Pad1)
- U10 pad 3: /Top PCB/ESP32/Motor PWM2 -> unconnected-(U10-Pad3)
- U10 pad 5: /Top PCB/Motors/Motor 2A -> unconnected-(U10-Pad5)
- U11 pad 1: Net-(R32-Pad2) -> /Top PCB/Power/VBAT
- U11 pad 3: +BATT -> /Top PCB/Power/VBAT
- U11 pad 4: /Top PCB/Power/Bat+VE -> unconnected-(U11-Pad4)
- U12 pad 1: Net-(R33-Pad2) -> Net-(R34-Pad2)
- U12 pad 3: /Line Sensor 5 Lower -> +BATT
- U12 pad 4: GND -> /Top PCB/Power/Bat+VE
- U2 pad 2: GND -> /Lower PCB GND
- U2 pad 4: GND -> /Lower PCB GND
- U3 pad 2: GND -> /Lower PCB GND
- U3 pad 4: GND -> /Lower PCB GND
- U4 pad 2: GND -> /Lower PCB GND
- U4 pad 4: GND -> /Lower PCB GND
- U5 pad 1: GND -> Net-(R7-Pad2)
- U5 pad 2: +3V3 -> /Lower PCB GND
- U5 pad 3: /Top PCB/ESP32/enable -> /Line Sensor 5 Lower
- U5 pad 4: unconnected-(U5-Pad4) -> /Lower PCB GND
- U6 pad 1: GND -> /Lower PCB 3V3
- U6 pad 2: Net-(R23-Pad2) -> /H-Bridge 1A Lower
- U6 pad 3: GND -> /H-Bridge 1B Lower
- U6 pad 4: /Top PCB/Power/PowerInInrush -> unconnected-(U6-Pad4)
- U6 pad 5: +BATT -> /Lower PCB/Motors/Motor 2A
- U6 pad 6: Net-(R21-Pad2) -> /Lower PCB GND
- U6 pad 7: Net-(R20-Pad1) -> /Lower PCB/Motors/Motor 1A
- U6 pad 8: /Top PCB/Power/PowerInInrush -> /Lower PCB 5V
- U6 pad 9: GND -> Net-(C6-Pad1)
- U8 pad 1: Net-(R26-Pad2) -> GND
- U8 pad 2: Net-(R27-Pad1) -> Net-(R28-Pad2)
- U8 pad 3: unconnected-(U8-Pad3) -> GND
- U8 pad 4: unconnected-(U8-Pad4) -> /Top PCB/Power/PowerInInrush
- U8 pad 5: unconnected-(U8-Pad5) -> +BATT
Routing:
- net GND: track 127.8 -> 0.00 mm, vias 53 -> 0
- net +BATT: track 123.4 -> 0.00 mm, vias 3 -> 0
- net +5V: track 116.1 -> 0.00 mm, vias 1 -> 0
- net /Top PCB/ESP32/5V Switched 1: track 106.4 -> 0.00 mm, vias 4 -> 0
- net /Line Sensor LEDs Lower: track 98.2 -> 0.00 mm
- net /Top PCB/ESP32/5V Switch Aux: track 72.9 -> 0.00 mm, vias 1 -> 0
- net /Line Sensor 4 Top: track 63.6 -> 0.00 mm
- net /Top PCB/ESP32/Bat I: track 57.3 -> 0.00 mm, vias 2 -> 0
- net /Top PCB/ESP32/Flash: track 56.7 -> 0.00 mm, vias 1 -> 0
- net /Line Sensor 3 Top: track 54.5 -> 0.00 mm
- net /Top PCB/ESP32/Reset: track 53.8 -> 0.00 mm, vias 1 -> 0
- net /Top PCB/ESP32/Motor PWM4: track 52.3 -> 0.00 mm, vias 2 -> 0
- net /Line Sensor 2 Top: track 51.2 -> 0.00 mm
- net /Top PCB/ESP32/Motor PWM3: track 50.5 -> 0.00 mm, vias 2 -> 0
- net /Sonar 5V Lower: track 46.0 -> 0.00 mm
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- added copper zone on B.Cu, net /Lower PCB 3V3
- added copper zone on F.Cu, net /Lower PCB GND
- removed copper zone on In2.Cu, net +3V3
- removed copper zone on In1.Cu, net GND
Other:
- board size 100 x 80 mm -> 100 x 180 mm
- copper layers 4 -> 2
- board text added: "Swarmbot Lower PCB Version 0.2"
- board text added: "Swarmbot Top PCB Version 0.2"
- board text added: "When re-importing changes to the PCB from the DXF file, the location is X 120 Y 50, and X 120 Y 150 on the layer Edge.Cuts. You will then need to un-group the imported pcb, and move some features to User.1 (center lines etc)"
- board text removed: "+5 VDC"
- board text removed: "Swarmbot Version 0.1"
- board text removed: "Swarmbot Version 0.2"
- board text removed: "Version 0.2"
- board text removed: "When re-importing changes to the PCB from the DXF file, the location is X 150 Y 100 on the layer Edge.Cuts. You will then need to un-group the imported pcb, and move some features to User.1 (center lines etc)"

Commit message: some pcb changes
Parts:
- added C27: 100pF, Capacitor_SMD:C_0805_2012Metric_Pad1.18x1.45mm_HandSolder, F.Cu at (144.3, 60.1)
- moved U12 226.9 mm to (224.0, 157.6)
- moved R27 225.0 mm to (247.9, 132.7)
- moved C13 225.0 mm to (238.3, 133.1)
- moved C14 225.0 mm to (232.3, 140.8)
- moved C26 225.0 mm to (239.7, 129.8)
- moved D4 225.0 mm to (243.1, 132.8)
- moved R17 225.0 mm to (247.0, 135.8)
- moved R18 225.0 mm to (242.3, 139.0)
- moved R23 225.0 mm to (237.1, 142.4)
- moved R32 225.0 mm to (242.3, 136.1)
- moved R26 215.9 mm to (234.6, 127.1)
- moved R31 198.1 mm to (206.9, 140.1)
- moved U8 194.9 mm to (206.6, 110.0)
- moved U9 189.8 mm to (197.2, 140.5)
- moved C7 181.2 mm to (154.2, 76.3), turned to 180 degrees
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Connections:
- J2 pad 6: /H-Bridge 2B Lower -> /H-Bridge 1A Lower
- J2 pad 8: /H-Bridge 1A Lower -> /H-Bridge 2B Lower
Routing:
- net /H-Bridge 2A Lower: track 0.00 -> 27.8 mm
- net /H-Bridge 2B Lower: track 0.00 -> 27.2 mm
- net /H-Bridge 1B Lower: track 0.00 -> 18.4 mm
- net /H-Bridge 1A Lower: track 0.00 -> 16.1 mm
- net /Lower PCB 3V3: track 0.00 -> 16.0 mm, vias 0 -> 2
- net Net-(C8-Pad1): track 0.00 -> 13.2 mm
- net /Lower PCB 5V: track 0.00 -> 7.92 mm, vias 0 -> 5
- net /Lower PCB GND: track 0.00 -> 5.49 mm, vias 0 -> 2
- net Net-(C7-Pad1): track 0.00 -> 5.06 mm
- net Net-(C6-Pad1): track 0.00 -> 4.67 mm
- net Net-(C8-Pad2): track 0.00 -> 3.67 mm
- net Net-(C7-Pad2): track 0.00 -> 3.09 mm
- added copper zone on B.Cu, net /Lower PCB 5V
- removed copper zone on B.Cu, net /Lower PCB 3V3
