File: Electronics/Motors.kicad_sch (KiCad schematic)
At the start: 7 parts, among them U6 MPC17531A

Commit message: del backups
Parts:
- renumbered C4 to C1, C5 to C2, C27 to C3, C6 to C4, C7 to C5, C8 to C6, U6 to U1
Changed lines of the file:
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@@
   (symbol (lib_id "Device:C_Small") (at 76.2 121.285 0) (unit 1)
     (in_bom yes) (on_board yes) (fields_autoplaced)
-    (property "Reference" "C4" (id 0) (at 78.74 120.0149 0)
+    (property "Reference" "C1" (id 0) (at 78.74 120.0149 0)
       (effects (font (size 1.27 1.27)) (justify left))
     )
@@
   (symbol (lib_id "Device:C_Small") (at 86.995 121.285 0) (unit 1)
     (in_bom yes) (on_board yes) (fields_autoplaced)
-    (property "Reference" "C5" (id 0) (at 89.535 120.0149 0)
+    (property "Reference" "C2" (id 0) (at 89.535 120.0149 0)
       (effects (font (size 1.27 1.27)) (justify left))
     )
@@
   (symbol (lib_id "Device:C_Small") (at 97.155 121.285 0) (unit 1)
     (in_bom yes) (on_board yes) (fields_autoplaced)
-    (property "Reference" "C27" (id 0) (at 99.695 120.0149 0)
+    (property "Reference" "C3" (id 0) (at 99.695 120.0149 0)
       (effects (font (size 1.27 1.27)) (justify left))
     )
@@
   (symbol (lib_id "Device:C_Small") (at 127.635 121.285 0) (unit 1)
     (in_bom yes) (on_board yes) (fields_autoplaced)
-    (property "Reference" "C6" (id 0) (at 130.175 120.0149 0)
+    (property "Reference" "C4" (id 0) (at 130.175 120.0149 0)
       (effects (font (size 1.27 1.27)) (justify left))
     )
@@
   (symbol (lib_id "Device:C_Small") (at 137.16 99.695 0) (unit 1)
     (in_bom yes) (on_board yes) (fields_autoplaced)
-    (property "Reference" "C7" (id 0) (at 139.7 98.4249 0)
+    (property "Reference" "C5" (id 0) (at 139.7 98.4249 0)
       (effects (font (size 1.27 1.27)) (justify left))
     )
@@
   (symbol (lib_id "Device:C_Small") (at 137.16 107.315 0) (unit 1)
     (in_bom yes) (on_board yes) (fields_autoplaced)
-    (property "Reference" "C8" (id 0) (at 139.7 106.0449 0)
+    (property "Reference" "C6" (id 0) (at 139.7 106.0449 0)
       (effects (font (size 1.27 1.27)) (justify left))
     )
@@
   (symbol (lib_id "MPC17531ATEJ - H Bridge:MPC17531A") (at 111.125 90.805 0) (unit 1)
     (in_bom yes) (on_board yes) (fields_autoplaced)
-    (property "Reference" "U6" (id 0) (at 112.395 120.65 0))
+    (property "Reference" "U1" (id 0) (at 112.395 120.65 0))
     (property "Value" "MPC17531A" (id 1) (at 112.395 123.19 0))
     (property "Footprint" "Package_SO:HTSSOP-20-1EP_4.4x6.5mm_P0.65mm_EP3.4x6.5mm_Mask2.75x3.43mm_ThermalVias_HandSolder" (id 2) (at 111.125 85.725 0)

Commit message: some changes were made
Other:
- company: (none) -> Squashed Fly
- title: (none) -> Swarmbot
